File: hw/bldc.kicad_pcb (KiCad board)
At the start: 2 copper layers, 177.8 x 101.6 mm, 287 parts, among them J1 Motor Phases, J2 Encoder1, J3 Encoder2, J4 USB_C_Receptacle, J5 USB_C_Receptacle, J6 Conn_ST_STDC14, J7 TC2070, Q1 2N7002K, Q2 2N7002, SW1 SW_Nidec_CAS-120A1, SW2 MCU Reset, SW3 User1, SW4 SW_Nidec_CAS-120A1, U1 CSD25402Q3A, U10 SIA400EDJ-T1-GE3, U11 SIA400EDJ-T1-GE3, U12 INA240A3PW, U13 SIA400EDJ-T1-GE3, U14 SIA400EDJ-T1-GE3, U15 INA240A3PW, U16 SIA400EDJ-T1-GE3, U17 SIA400EDJ-T1-GE3, U18 INA240A3PW, U2 CSD25402Q3A, U3 INA180A2, U4 CYPD3177-24LQ, U5 LMR50410, U6 LD1117S33TR_SOT223, U7 TPS2116DRL, U8 STSPIN32G4, U9 BNO055, Y1 25MHz

Commit message: some layout
Parts:
- moved C1 219.5 mm to (26.7, 38.7), turned to 90 degrees
- moved C2 214.8 mm to (29.2, 38.7), turned to -90 degrees
- moved D1 201.8 mm to (19.1, 52.7)
- moved C6 200.7 mm to (52.1, 24.1), turned to 180 degrees
- moved R18 192.4 mm to (32.4, 50.2)
- moved Q1 187.2 mm to (28.6, 48.9), turned to 180 degrees
- moved R19 184.7 mm to (29.2, 43.8), turned to 180 degrees
- moved R20 183.6 mm to (32.4, 48.3)
- moved C12 183.5 mm to (43.8, 37.5)
- moved R17 179.5 mm to (30.5, 30.5)
- moved C8 179.0 mm to (61.6, -3.17)
- moved R12 178.0 mm to (30.5, 29.2)
- moved U5 176.4 mm to (43.8, 40.0)
- moved R16 175.8 mm to (58.6, -6.99)
- moved R3 175.7 mm to (30.5, 33.0)
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Other:
- copper layers 2 -> 4
- board text added: "12V"
- board text added: "20V"

Commit message: More layout
Parts:
- removed the R46 at (249.7, 81.7)
- added C48: 4.7uF, Capacitor_SMD:C_0805_2012Metric, F.Cu at (59.1, 90.2)
- added Dial_Scale**: GM6208, pcs_lib:GM6208, F.Cu at (142.2, 71.1)
- added Dial_Scale**: GM2804_dial, pcs_lib:GM2804_dial, F.Cu at (33.0, 104.1)
- added NT10: NetTie_2, NetTie:NetTie-2_SMD_Pad0.5mm, F.Cu at (44.2, 34.4)
- added NT11: NetTie_2, NetTie:NetTie-2_SMD_Pad0.5mm, F.Cu at (47.2, 34.4)
- added kibuzzard-69046065: G***, kibuzzard-69046065, F.Cu at (136.5, 27.3)
- added kibuzzard-6904608C: G***, kibuzzard-6904608C, F.Cu at (186.1, 64.1)
- added kibuzzard-690460A4: G***, kibuzzard-690460A4, F.Cu at (149.9, 114.9)
- added kibuzzard-690460EC: G***, kibuzzard-690460EC, F.Cu at (98.4, 74.9)
- added kibuzzard-690461AA: G***, kibuzzard-690461AA, B.Cu at (113.7, 114.3)
- added kibuzzard-69056F08: G***, kibuzzard-69056F08, F.Cu at (29.2, 55.9)
- added kibuzzard-69056F8E: G***, kibuzzard-69056F8E, F.Cu at (26.0, 60.3)
- added kibuzzard-69056FD5: G***, kibuzzard-69056FD5, F.Cu at (26.0, 64.8)
- added kibuzzard-6905703C: G***, kibuzzard-6905703C, F.Cu at (32.4, 69.2)
- added kibuzzard-690572FD: G***, kibuzzard-690572FD, F.Cu at (36.8, 74.9)
- added kibuzzard-69057344: G***, kibuzzard-69057344, F.Cu at (169.5, 109.2)
- D10, D11, D12, D13, D14, D15, D16, D17, D18, D19, D20, D21, D22, D23, D24, D25, D26, D27, D28, D29, D30, D31, D32, D33, D34, D35, D36, D37, D38, D39, D40, D41, D42, D43, D8, D9: footprint LED_SMD:LED_SK6805_PLCC4_2.4x2.7mm_P1.3mm -> pcs_lib:LED_SK6805_PLCC4_2.4x2.7mm_P1.3mm
- moved C17 221.7 mm to (59.1, 37.5), turned to 90 degrees
- moved SW2 212.4 mm to (23.5, 74.9)
- moved C22 208.7 mm to (25.9, 25.4), turned to -90 degrees
- moved R39 207.2 mm to (59.1, 23.5)
- moved R43 207.0 mm to (59.1, 26.0)
- moved R40 207.0 mm to (59.1, 22.2)
- moved R42 205.8 mm to (59.1, 24.8)
- moved D3 202.3 mm to (19.1, 64.8), turned to -90 degrees
- moved NT3 200.6 mm to (77.5, 105.4), turned to 90 degrees
- moved C45 200.0 mm to (59.1, 97.8), turned to 180 degrees
- moved NT4 198.7 mm to (76.8, 107.3), turned to 90 degrees
- moved C26 198.3 mm to (19.1, 74.9), turned to 90 degrees
- moved C18 198.1 mm to (69.8, 34.9), turned to -90 degrees
- moved D2 197.7 mm to (19.1, 60.3), turned to -90 degrees
- moved D4 196.9 mm to (19.1, 69.2), turned to -90 degrees
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- renumbered C99 to C100, C100 to C101, C101 to C102, C102 to C103, C103 to C104, C104 to C105, C48 to C49, C49 to C50, C50 to C51, C51 to C52, C52 to C53, C53 to C54, C54 to C55, C55 to C56, C56 to C57, C57 to C58, C58 to C59, C59 to C60, C60 to C61, C61 to C62, C62 to C63, C63 to C64, C64 to C65, C65 to C66, C66 to C67, C67 to C68, C68 to C69, C69 to C70, C70 to C71, C71 to C72, C72 to C73, C73 to C74, C74 to C75, C75 to C76, C76 to C77, C77 to C78, C78 to C79, C79 to C80, C80 to C81, C81 to C82, C82 to C83, C83 to C84, C84 to C85, C85 to C86, C86 to C87, C87 to C88, C88 to C89, C89 to C90, C90 to C91, C91 to C92, C92 to C93, C93 to C94, C94 to C95, C95 to C96, C96 to C97, C97 to C98, C98 to C99, R29 to R28, R28 to R29, R31 to R30, R30 to R31, R47 to R45, R48 to R46, R49 to R47, R50 to R48, R51 to R49, R52 to R50, R53 to R51, R54 to R52, R55 to R53, R56 to R54, R57 to R55, R58 to R56, R59 to R57, R60 to R58, R61 to R59, R62 to R60, R63 to R61, R64 to R62, R65 to R63, R66 to R64, R67 to R65, R68 to R66, R69 to R67, R70 to R68, R71 to R69, R72 to R70
Connections:
- C26 pad 2: 3V3 -> /micro/nRST
- C27 pad 2: 3V3 -> /micro/USER_BTN_1
- C28 pad 2: 3V3 -> /micro/MCU_BOOT0/I2C_SCL
- C3 pad 1: Net-(U1-G) -> /input-power/VBUS_FET_GATE
- C4 pad 1: /input-power/VBUS_ISENSE_HI -> /input-power/VDC_OUT
- C4 pad 2: Net-(U1-G) -> /input-power/VBUS_FET_GATE
- D2 pad 1: Net-(D2-K) -> GND
- D2 pad 2: 5V0_BUCK -> Net-(D2-A)
- D3 pad 1: Net-(D3-K) -> GND
- D3 pad 2: 3V3 -> Net-(D3-A)
- D4 pad 1: Net-(D4-K) -> GND
- D4 pad 2: MCU_USB_VBUS -> Net-(D4-A)
- R1 pad 1: /input-power/VBUS_ISENSE_HI -> /input-power/VDC_OUT
- R10 pad 2: Net-(U1-G) -> /input-power/VBUS_FET_GATE
- R22 pad 1: Net-(D2-K) -> 5V0_BUCK
- R22 pad 2: GND -> Net-(D2-A)
- R28 pad 1: Net-(D3-K) -> 3V3
- R28 pad 2: GND -> Net-(D3-A)
- R3 pad 2: Net-(U1-G) -> /input-power/VBUS_FET_GATE
- R30 pad 1: Net-(D4-K) -> MCU_USB_VBUS
- R30 pad 2: GND -> Net-(D4-A)
- R4 pad 2: Net-(U1-G) -> /input-power/VBUS_FET_GATE
- R5 pad 1: Net-(U1-S) -> /input-power/VBUS_FET_SW
- R5 pad 2: Net-(U1-G) -> /input-power/VBUS_FET_GATE
- R6 pad 1: Net-(U1-S) -> /input-power/VBUS_FET_SW
- R6 pad 2: Net-(U1-G) -> /input-power/VBUS_FET_GATE
- R9 pad 2: Net-(U1-G) -> /input-power/VBUS_FET_GATE
- U1 pad 1: (no net) -> VBUS_IN
- U1 pad 2: (no net) -> VBUS_IN
- U1 pad 3: (no net) -> VBUS_IN
- U1 pad 4: (no net) -> /input-power/VBUS_FET_GATE
- U1 pad 5: (no net) -> /input-power/VBUS_FET_SW
- U2 pad 1: /input-power/VBUS_ISENSE_HI -> /input-power/VDC_OUT
- U2 pad 2: /input-power/VBUS_ISENSE_HI -> /input-power/VDC_OUT
- U2 pad 3: /input-power/VBUS_ISENSE_HI -> /input-power/VDC_OUT
- U2 pad 4: Net-(U1-G) -> /input-power/VBUS_FET_GATE
- U2 pad 5: Net-(U1-S) -> /input-power/VBUS_FET_SW
- U3 pad 4: VBUS -> /input-power/VBUS_ISENSE_LOW
- U4 pad 11: /input-power/VBUS_ISENSE_HI -> /input-power/VDC_OUT
Routing:
- net GND: track 0.00 -> 72.5 mm, vias 0 -> 46
- net MCU_USB_VBUS: track 0.00 -> 55.6 mm
- net Net-(SW1-B): track 0.00 -> 26.6 mm, vias 0 -> 2
- net /micro/MCU_BOOT0/I2C_SCL: track 0.00 -> 26.5 mm, vias 0 -> 2
- net /micro/USB_P: track 0.00 -> 24.9 mm
- net /micro/USB_N: track 0.00 -> 24.1 mm
- net /input-power/VDC_OUT: track 0.00 -> 22.6 mm, vias 0 -> 2
- net /input-power/CC1: track 0.00 -> 22.2 mm
- net /micro/USART1_RX: track 0.00 -> 19.0 mm
- net /input-power/CC2: track 0.00 -> 17.6 mm
- net Net-(U4-FLIP): track 0.00 -> 16.8 mm, vias 0 -> 2
- net 3V3: track 0.00 -> 16.7 mm, vias 0 -> 23
- net /micro/USART1_TX: track 0.00 -> 15.4 mm
- net 5V0: track 0.00 -> 14.5 mm, vias 0 -> 3
- net VBUS: track 0.00 -> 13.6 mm, vias 0 -> 3
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- added copper zone on F.Cu, net /input-power/VBUS_FET_GATE
- added copper zone on F.Cu, net /input-power/VBUS_FET_SW
- added copper zone on F.Cu, net /input-power/VDC_OUT
- added copper zone on F.Cu, net 3V3
- added copper zone on In2.Cu, net 3V3
- added copper zone on B.Cu, net 5V0
- added copper zone on F.Cu, net 5V0_BUCK
- added copper zone on In1.Cu, net GND
- added copper zone on F.Cu, net MCU_USB_VBUS
- added copper zone on B.Cu, net VBUS
- added copper zone on F.Cu, net VBUS
- added copper zone on F.Cu, net VBUS_IN
- added copper zone on F.Cu, net VCC
- added copper zone on F.Cu, net VDDD
Other:
- outline, holes or cut-outs redrawn

Commit message: layout 'finished' need to start double checking everything
Parts:
- removed the NT7 at (111.1, 5.71)
- removed the NT8 at (127.6, 8.45)
- removed NT9: NetTie_2, NetTie:NetTie-2_SMD_Pad0.5mm
- removed the R45 at (73.7, 58.4)
- added R43: 0Ω, Resistor_SMD:R_0402_1005Metric, F.Cu at (67.9, 60.3)
- added TP17: RGB_DIN_5V0, TestPoint:TestPoint_Pad_1.0x1.0mm, F.Cu at (61.6, 60.3)
- added kibuzzard-6976CBB1: G***, kibuzzard-6976CBB1, F.Cu at (128.0, 112.4)
- TP6: value 5V0_VSENSE -> VBUS
- TP8: value 5V0_VSENSE -> 5V0
- TP9: value 5V0_VSENSE -> 3V3
- moved R64 124.5 mm to (66.0, 97.2)
- moved C97 122.4 mm to (66.0, 95.9), turned to 180 degrees
- moved C98 112.4 mm to (60.3, 100.3), turned to -90 degrees
- moved C95 109.7 mm to (62.2, 100.3), turned to -90 degrees
- moved U14 108.3 mm to (63.5, 85.1), turned to 0 degrees
- moved R63 108.1 mm to (62.2, 88.3), turned to 180 degrees
- moved U15 107.4 mm to (62.2, 94.0), turned to -90 degrees
- moved C96 107.0 mm to (64.1, 100.3), turned to -90 degrees
- moved R57 105.4 mm to (85.1, 88.9)
- moved D45 104.9 mm to (61.0, 85.1), turned to 90 degrees
- moved C100 104.6 mm to (89.5, 81.3)
- moved R67 104.6 mm to (89.5, 80.0)
- moved U17 103.8 mm to (72.4, 74.3)
- moved U11 103.7 mm to (72.4, 91.4)
- moved U13 103.5 mm to (63.5, 81.9), turned to 0 degrees
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- renumbered NT10 to NT1, NT11 to NT2, NT1 to NT3, NT2 to NT4, NT3 to NT5, NT4 to NT6, NT5 to NT7, NT6 to NT8, R43 to R44, R44 to R45, R45 to R46, R46 to R47, R47 to R48, R48 to R49, R49 to R50, R50 to R51, R51 to R52, R52 to R53, R53 to R54, R54 to R55, R55 to R56, R56 to R57, R57 to R58, R58 to R59, R59 to R60, R60 to R61, R61 to R62, R62 to R63, R63 to R64, R64 to R65, R65 to R66, R66 to R67, R67 to R68, R68 to R69, R69 to R70, R70 to R71, TP17 to TP18, TP18 to TP19, TP19 to TP20, TP20 to TP21, TP21 to TP22, TP22 to TP23
Connections:
- C100 pad 2: /micro/PHASE_W_ISENSE -> /micro/OPAMP3_VINP
- C101 pad 1: /micro/PHASE_W_ISENSE -> /micro/OPAMP3_VINP
- C104 pad 2: /micro/OPAMP3_VINP -> /micro/PHASE_W_ISENSE
- C93 pad 2: /micro/PHASE_V_ISENSE -> /micro/OPAMP2_VINP
- C94 pad 1: /micro/PHASE_V_ISENSE -> /micro/OPAMP2_VINP
- C97 pad 2: /micro/OPAMP2_VINP -> /micro/PHASE_V_ISENSE
- NT3 pad 1: /micro/SPI3_MOSI -> /micro/RGB_DIN
- NT3 pad 2: /micro/RGB_DIN -> /micro/SPI3_MOSI
- R60 pad 2: /micro/PHASE_V_ISENSE -> /micro/OPAMP2_VINP
- R62 pad 1: /micro/PHASE_V_ISENSE -> /micro/OPAMP2_VINP
- R64 pad 2: /micro/OPAMP2_VINP -> /micro/PHASE_V_ISENSE
- R67 pad 2: /micro/PHASE_W_ISENSE -> /micro/OPAMP3_VINP
- R69 pad 1: /micro/PHASE_W_ISENSE -> /micro/OPAMP3_VINP
- R71 pad 2: /micro/OPAMP3_VINP -> /micro/PHASE_W_ISENSE
- U12 pad 6: Net-(U12-REF2) -> 3V3
- U15 pad 6: Net-(U15-REF2) -> 3V3
- U18 pad 6: Net-(U18-REF2) -> 3V3
Routing:
- net /micro/nRST: track 7.53 -> 189.3 mm, vias 0 -> 4
- net /micro/USER_BTN_1: track 0.00 -> 165.3 mm, vias 0 -> 4
- net GND: track 72.5 -> 209.5 mm, vias 46 -> 259
- net 5V0: track 14.5 -> 148.6 mm, vias 3 -> 41
- net Net-(U10-G): track 0.00 -> 118.2 mm
- net /micro/ENCODER_1_CS: track 0.00 -> 109.5 mm
- net /micro/MCU_BOOT0/I2C_SCL: track 26.5 -> 134.9 mm, vias 2 -> 5
- net /micro/ENCODER_2_CS: track 0.00 -> 102.7 mm, vias 0 -> 2
- net /micro/SPI1_SCK: track 0.00 -> 101.3 mm
- net Net-(D44-K): track 0.00 -> 100.9 mm
- net /micro/SPI1_MISO: track 0.00 -> 99.9 mm
- net /micro/SPI1_MOSI: track 0.00 -> 98.8 mm
- net Net-(U16-G): track 0.00 -> 97.0 mm, vias 0 -> 2
- net Net-(U13-G): track 0.00 -> 96.5 mm, vias 0 -> 2
- net /micro/I2C_SDA: track 10.7 -> 104.9 mm, vias 2 -> 4
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- added copper zone on F.Cu, net /motor-phases/PHASE_U
- added copper zone on F.Cu, net /motor-phases/PHASE_V
- added copper zone on F.Cu, net /motor-phases/PHASE_W
- added copper zone on F.Cu, net GND
- added copper zone on F.Cu, net Net-(U11-S)
- added copper zone on F.Cu, net Net-(U14-S)
- added copper zone on F.Cu, net Net-(U17-S)

Commit message: finalized / checked design
Parts:
- removed R14, R15: 2.4k, Resistor_SMD:R_0402_1005Metric
- added NT10: NetTie_2, NetTie:NetTie-2_SMD_Pad0.5mm, B.Cu at (87.6, 84.5)
- added NT12: NetTie_2, NetTie:NetTie-2_SMD_Pad0.5mm, B.Cu at (87.6, 81.9)
- added NT9: NetTie_2, NetTie:NetTie-2_SMD_Pad0.5mm, B.Cu at (87.6, 79.4)
Connections:
- net /micro/ENCODER_1_CS renamed /micro/ENC_SPI_CS0
- net /micro/ENCODER_2_CS renamed /micro/ENC_SPI_CS1
- net /micro/ENCODER_SPI_MISO renamed /micro/ENC_SPI_MISO
- net /micro/ENCODER_SPI_MOSI renamed /micro/ENC_SPI_MOSI
- net /micro/ENCODER_SPI_SCK renamed /micro/ENC_SPI_SCK
- C100 pad 2: /micro/OPAMP3_VINP -> /micro/PHASE_W_VSENSE
- C101 pad 1: /micro/OPAMP3_VINP -> /micro/PHASE_W_VSENSE
- C86 pad 2: /micro/OPAMP1_VINP -> /micro/PHASE_U_VSENSE
- C87 pad 1: /micro/OPAMP1_VINP -> /micro/PHASE_U_VSENSE
- C93 pad 2: /micro/OPAMP2_VINP -> /micro/PHASE_V_VSENSE
- C94 pad 1: /micro/OPAMP2_VINP -> /micro/PHASE_V_VSENSE
- R53 pad 2: /micro/OPAMP1_VINP -> /micro/PHASE_U_VSENSE
- R55 pad 1: /micro/OPAMP1_VINP -> /micro/PHASE_U_VSENSE
- R60 pad 2: /micro/OPAMP2_VINP -> /micro/PHASE_V_VSENSE
- R62 pad 1: /micro/OPAMP2_VINP -> /micro/PHASE_V_VSENSE
- R67 pad 2: /micro/OPAMP3_VINP -> /micro/PHASE_W_VSENSE
- R69 pad 1: /micro/OPAMP3_VINP -> /micro/PHASE_W_VSENSE
Routing:
- net VBUS: track 59.6 -> 29.2 mm, vias 21 -> 26
- net /micro/MCU_BOOT0/I2C_SCL: track 134.9 -> 122.9 mm, vias 5 -> 4
- net /micro/I2C_SDA: track 104.9 -> 96.4 mm, vias 4 -> 3
- net /micro/OPAMP3_VINP: track 41.5 -> 33.9 mm, vias 2 -> 1
- net /micro/OPAMP2_VINP: track 42.7 -> 35.1 mm, vias 2 -> 1
- net /micro/OPAMP1_VINP: track 45.8 -> 38.3 mm, vias 2 -> 1
- net /micro/PHASE_V_VSENSE: track 0.00 -> 6.56 mm, vias 0 -> 1
- net /micro/PHASE_W_VSENSE: track 0.00 -> 6.55 mm, vias 0 -> 1
- net /micro/PHASE_U_VSENSE: track 0.00 -> 6.55 mm, vias 0 -> 1
- net VBUS_IN: track 9.21 -> 11.4 mm
- net 3V3: track 39.2 -> 37.3 mm
- net Net-(U4-FLIP): track 17.3 -> 15.9 mm
- net Net-(SW1-B): track 33.8 -> 35.1 mm
- net Net-(Q1-G): track 18.7 -> 19.2 mm
- net GND: vias 259 -> 264
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Other:
- board text added: "5V0"
- board text added: "CS0"
- board text added: "CS1"
- board text added: "GND"
- board text added: "MISO"
- board text added: "MOSI"
- board text added: "SCK"
