File: hw/bldc.kicad_sch (KiCad schematic)
At the start: 3 parts, among them J1 Motor Phases, J2 Encoder1, J3 Encoder2

Commit message: finalized / checked design
Parts:
- J1: MPN (none) -> S3B-XH-A(LF)(SN)
- J2, J3: MPN (none) -> S6B-PH-K-S(LF)(SN)
Changed lines of the file:
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@@
+			)
+		)
+		(property "MPN" "S3B-XH-A(LF)(SN)"
+			(at 0 0 0)
+			(effects
+				(font
+					(size 1.27 1.27)
+				)
+				(hide yes)
 			)
 		)
@@
 			)
 		)
+		(property "MPN" "S6B-PH-K-S(LF)(SN)"
+			(at 0 0 0)
+			(effects
+				(font
+					(size 1.27 1.27)
+				)
+				(hide yes)
+			)
+		)
 		(pin "5"
 		)
@@
 			(effects
 				(font
+					(size 1.27 1.27)
+				)
+				(hide yes)
+			)
+		)
+		(property "MPN" "S6B-PH-K-S(LF)(SN)"
+			(at 0 0 0)
+			(effects
+				(font
