File: hw/half_bridge.kicad_sch (KiCad schematic)
At the start: 19 parts, among them U10 SIA400EDJ-T1-GE3, U11 SIA400EDJ-T1-GE3, U12 INA240A3PW

Commit message: More layout
Parts:
- renumbered C84 to C85, C85 to C86, C86 to C87, C87 to C88, C88 to C89, C89 to C90, C90 to C91, R52 to R50, R53 to R51, R54 to R52, R55 to R53, R56 to R54, R57 to R55, R58 to R56

Commit message: layout 'finished' need to start double checking everything
Parts:
- removed NT7: NetTie_2, NetTie:NetTie-2_SMD_Pad0.5mm, symbol Device:NetTie_2
- renumbered R50 to R51, R51 to R52, R52 to R53, R53 to R54, R54 to R55, R55 to R56, R56 to R57
Connections:
- net 3V3: now also U12.6 (REF2)
Changed lines of the file:
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@@
 	(wire
 		(pts
-			(xy 139.7 137.16) (xy 135.89 137.16)
+			(xy 135.89 137.16) (xy 148.59 137.16)
 		)
 		(stroke
@@
 		(pts
 			(xy 165.1 107.95) (xy 165.1 109.22)
-		)
-		(stroke
-			(width 0)
-			(type default)
-		)
-	)
-	(wire
-		(pts
-			(xy 144.78 137.16) (xy 148.59 137.16)
 		)
 		(stroke
@@
 		(on_board yes)
 		(dnp no)
-		(property "Reference" "R54"
+		(property "Reference" "R55"
 			(at 148.336 76.2 0)
 			(effects
@@
 			(project "bldc"
 				(path "/fdf9474f-66c9-4c2c-9436-f3125b555611/066314e2-1f8c-41a2-8da1-0e67cde6d8c9/04e27305-6622-4569-b655-167b284d3f8d"
-					(reference "R61")
+					(reference "R62")
 					(unit 1)
 				)
 				(path "/fdf9474f-66c9-4c2c-9436-f3125b555611/066314e2-1f8c-41a2-8da1-0e67cde6d8c9/28abe682-412f-4f29-a286-a025fbee515c"
-					(reference "R68")
+					(reference "R69")
 					(unit 1)
 				)
 				(path "/fdf9474f-66c9-4c2c-9436-f3125b555611/066314e2-1f8c-41a2-8da1-0e67cde6d8c9/e94933e5-d530-4653-91dd-3749c1487490"
-					(reference "R54")
+					(reference "R55")
 					(unit 1)
 				)
@@
 		(dnp no)
 		(fields_autoplaced yes)
-		(property "Reference" "R55"
+		(property "Reference" "R56"
 			(at 124.46 118.1099 0)
 			(effects
@@
 			(project "bldc"
 				(path "/fdf9474f-66c9-4c2c-9436-f3125b555611/066314e2-1f8c-41a2-8da1-0e67cde6d8c9/04e27305-6622-4569-b655-167b284d3f8d"
-					(reference "R62")
+					(reference "R63")
 					(unit 1)
 				)
 				(path "/fdf9474f-66c9-4c2c-9436-f3125b555611/066314e2-1f8c-41a2-8da1-0e67cde6d8c9/28abe682-412f-4f29-a286-a025fbee515c"
-					(reference "R69")
+					(reference "R70")
 					(unit 1)
 				)
 				(path "/fdf9474f-66c9-4c2c-9436-f3125b555611/066314e2-1f8c-41a2-8da1-0e67cde6d8c9/e94933e5-d530-4653-91dd-3749c1487490"
-					(reference "R55")
+					(reference "R56")
 					(unit 1)
 				)
@@
 		(dnp no)
 		(fields_autoplaced yes)
-		(property "Reference" "R50"
+		(property "Reference" "R51"
 			(at 95.25 49.53 90)
 			(effects
@@
 			(project "bldc"
 				(path "/fdf9474f-66c9-4c2c-9436-f3125b555611/066314e2-1f8c-41a2-8da1-0e67cde6d8c9/04e27305-6622-4569-b655-167b284d3f8d"
-					(reference "R57")
+					(reference "R58")
 					(unit 1)
 				)
 				(path "/fdf9474f-66c9-4c2c-9436-f3125b555611/066314e2-1f8c-41a2-8da1-0e67cde6d8c9/28abe682-412f-4f29-a286-a025fbee515c"
-					(reference "R64")
+					(reference "R65")
 					(unit 1)
 				)
 				(path "/fdf9474f-66c9-4c2c-9436-f3125b555611/066314e2-1f8c-41a2-8da1-0e67cde6d8c9/e94933e5-d530-4653-91dd-3749c1487490"
-					(reference "R50")
+					(reference "R51")
 					(unit 1)
 				)
@@
 		(dnp no)
 		(fields_autoplaced yes)
-		(property "Reference" "R52"
+		(property "Reference" "R53"
 			(at 148.59 67.3099 0)
 			(effects
@@
 			(project "bldc"
 				(path "/fdf9474f-66c9-4c2c-9436-f3125b555611/066314e2-1f8c-41a2-8da1-0e67cde6d8c9/04e27305-6622-4569-b655-167b284d3f8d"
-					(reference "R59")
+					(reference "R60")
 					(unit 1)
 				)
 				(path "/fdf9474f-66c9-4c2c-9436-f3125b555611/066314e2-1f8c-41a2-8da1-0e67cde6d8c9/28abe682-412f-4f29-a286-a025fbee515c"
-					(reference "R66")
+					(reference "R67")
 					(unit 1)
 				)
 				(path "/fdf9474f-66c9-4c2c-9436-f3125b555611/066314e2-1f8c-41a2-8da1-0e67cde6d8c9/e94933e5-d530-4653-91dd-3749c1487490"
-					(reference "R52")
+					(reference "R53")
 					(unit 1)
 				)
@@
 		(on_board yes)
 		(dnp no)
-		(property "Reference" "R51"
+		(property "Reference" "R52"
 			(at 114.3 65.278 90)
 			(effects
@@
 			(project "bldc"
 				(path "/fdf9474f-66c9-4c2c-9436-f3125b555611/066314e2-1f8c-41a2-8da1-0e67cde6d8c9/04e27305-6622-4569-b655-167b284d3f8d"
-					(reference "R58")
+					(reference "R59")
 					(unit 1)
 				)
 				(path "/fdf9474f-66c9-4c2c-9436-f3125b555611/066314e2-1f8c-41a2-8da1-0e67cde6d8c9/28abe682-412f-4f29-a286-a025fbee515c"
-					(reference "R65")
+					(reference "R66")
 					(unit 1)
 				)
 				(path "/fdf9474f-66c9-4c2c-9436-f3125b555611/066314e2-1f8c-41a2-8da1-0e67cde6d8c9/e94933e5-d530-4653-91dd-3749c1487490"
-					(reference "R51")
+					(reference "R52")
 					(unit 1)
 				)
@@
 		(dnp no)
 		(fields_autoplaced yes)
-		(property "Reference" "R53"
+		(property "Reference" "R54"
 			(at 95.25 67.31 90)
 			(effects
@@
 			(project "bldc"
 				(path "/fdf9474f-66c9-4c2c-9436-f3125b555611/066314e2-1f8c-41a2-8da1-0e67cde6d8c9/04e27305-6622-4569-b655-167b284d3f8d"
-					(reference "R60")
+					(reference "R61")
 					(unit 1)
 				)
 				(path "/fdf9474f-66c9-4c2c-9436-f3125b555611/066314e2-1f8c-41a2-8da1-0e67cde6d8c9/28abe682-412f-4f29-a286-a025fbee515c"
-					(reference "R67")
+					(reference "R68")
 					(unit 1)
 				)
 				(path "/fdf9474f-66c9-4c2c-9436-f3125b555611/066314e2-1f8c-41a2-8da1-0e67cde6d8c9/e94933e5-d530-4653-91dd-3749c1487490"
-					(reference "R53")
+					(reference "R54")
 					(unit 1)
 				)
@@
 	)
 	(symbol
-		(lib_id "Device:NetTie_2")
-		(at 142.24 137.16 0)
-		(unit 1)
-		(exclude_from_sim no)
-		(in_bom no)
-		(on_board yes)
-		(dnp no)
-		(fields_autoplaced yes)
-		(property "Reference" "NT7"
-			(at 142.24 132.08 0)
-			(effects
-				(font
-					(size 1.27 1.27)
-				)
-				(hide yes)
-			)
-		)
-		(property "Value" "NetTie_2"
-			(at 142.24 134.62 0)
-			(effects
-				(font
-					(size 1.27 1.27)
-				)
-				(hide yes)
-			)
-		)
-		(property "Footprint" "NetTie:NetTie-2_SMD_Pad0.5mm"
-			(at 142.24 137.16 0)
-			(effects
-				(font
-					(size 1.27 1.27)
-				)
-				(hide yes)
-			)
-		)
-		(property "Datasheet" "~"
-			(at 142.24 137.16 0)
-			(effects
-				(font
-					(size 1.27 1.27)
-				)
-				(hide yes)
-			)
-		)
-		(property "Description" "Net tie, 2 pins"
-			(at 142.24 137.16 0)
-			(effects
-				(font
-					(size 1.27 1.27)
-				)
-				(hide yes)
-			)
-		)
-		(pin "2"
-		)
-		(pin "1"
-		)
-		(instances
-			(project "bldc"
-				(path "/fdf9474f-66c9-4c2c-9436-f3125b555611/066314e2-1f8c-41a2-8da1-0e67cde6d8c9/04e27305-6622-4569-b655-167b284d3f8d"
-					(reference "NT8")
-					(unit 1)
-				)
-				(path "/fdf9474f-66c9-4c2c-9436-f3125b555611/066314e2-1f8c-41a2-8da1-0e67cde6d8c9/28abe682-412f-4f29-a286-a025fbee515c"
-					(reference "NT9")
-					(unit 1)
-				)
-				(path "/fdf9474f-66c9-4c2c-9436-f3125b555611/066314e2-1f8c-41a2-8da1-0e67cde6d8c9/e94933e5-d530-4653-91dd-3749c1487490"
-					(reference "NT7")
-					(unit 1)
-				)
-			)
-		)
-	)
-	(symbol
 		(lib_id "Device:C_Small")
 		(at 160.02 104.14 0)
@@
 		(on_board yes)
 		(dnp no)
-		(property "Reference" "R56"
+		(property "Reference" "R57"
 			(at 162.56 118.872 90)
 			(effects
@@
 			(project "bldc"
 				(path "/fdf9474f-66c9-4c2c-9436-f3125b555611/066314e2-1f8c-41a2-8da1-0e67cde6d8c9/04e27305-6622-4569-b655-167b284d3f8d"
-					(reference "R63")
+					(reference "R64")
 					(unit 1)
 				)
 				(path "/fdf9474f-66c9-4c2c-9436-f3125b555611/066314e2-1f8c-41a2-8da1-0e67cde6d8c9/28abe682-412f-4f29-a286-a025fbee515c"
-					(reference "R70")
+					(reference "R71")
 					(unit 1)
 				)
 				(path "/fdf9474f-66c9-4c2c-9436-f3125b555611/066314e2-1f8c-41a2-8da1-0e67cde6d8c9/e94933e5-d530-4653-91dd-3749c1487490"
-					(reference "R56")
-					(unit 1)
-				)
+					(reference "R57")
+					(unit 1)
+				)

Commit message: finalized / checked design
Parts:
- C85, C88: MPN (none) -> CL21A475KAQNNNE
- C86: MPN (none) -> GJM1555C1H2R7BB01D
- C87: MPN (none) -> CL05C330JB5NNNC
- C89, C91: MPN (none) -> CL05B104KB54PNC
- C90: MPN (none) -> GCM155R71H122KA37D
- D44: MPN (none) -> BAT41KFILM
- R51, R54: MPN (none) -> RC0402FR-0733RL
- R52: MPN (none) -> RC0402FR-070RL
- R53: MPN (none) -> RC0402FR-07274KL
- R55: MPN (none) -> RC0402FR-0722K1L
- R56: MPN (none) -> PA1206FRF470R001L
- R57: MPN (none) -> RC0402FR-071KL
- U10, U11: MPN (none) -> SIA400EDJ-T1-GE3
- U12: MPN (none) -> INA240A3PW
Changed lines of the file:
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@@
+			)
+		)
+		(property "MPN" "RC0402FR-0722K1L"
+			(at 0 0 0)
+			(effects
+				(font
+					(size 1.27 1.27)
+				)
+				(hide yes)
 			)
 		)
@@
 			)
 		)
+		(property "MPN" "PA1206FRF470R001L"
+			(at 0 0 0)
+			(effects
+				(font
+					(size 1.27 1.27)
+				)
+				(hide yes)
+			)
+		)
 		(pin "2"
 		)
@@
 			)
 		)
+		(property "MPN" "RC0402FR-0733RL"
+			(at 0 0 0)
+			(effects
+				(font
+					(size 1.27 1.27)
+				)
+				(hide yes)
+			)
+		)
 		(pin "1"
 		)
@@
 			)
 		)
+		(property "MPN" "CL05B104KB54PNC"
+			(at 0 0 0)
+			(effects
+				(font
+					(size 1.27 1.27)
+				)
+				(hide yes)
+			)
+		)
 		(pin "1"
 		)
@@
 			)
 		)
+		(property "MPN" "BAT41KFILM"
+			(at 0 0 0)
+			(effects
+				(font
+					(size 1.27 1.27)
+				)
+				(hide yes)
+			)
+		)
 		(pin "2"
 		)
@@
 			)
 		)
+		(property "MPN" "CL05B104KB54PNC"
+			(at 0 0 0)
+			(effects
+				(font
+					(size 1.27 1.27)
+				)
+				(hide yes)
+			)
+		)
 		(pin "1"
 		)
@@
 			)
 		)
+		(property "MPN" "GCM155R71H122KA37D"
+			(at 0 0 0)
+			(effects
+				(font
+					(size 1.27 1.27)
+				)
+				(hide yes)
+			)
+		)
 		(pin "2"
 		)
@@
 			)
 		)
+		(property "MPN" "SIA400EDJ-T1-GE3"
+			(at 0 0 0)
+			(effects
+				(font
+					(size 1.27 1.27)
+				)
+				(hide yes)
+			)
+		)
 		(pin "1"
 		)
@@
 			)
 		)
+		(property "MPN" "CL21A475KAQNNNE"
+			(at 0 0 0)
+			(effects
+				(font
+					(size 1.27 1.27)
+				)
+				(hide yes)
+			)
+		)
 		(pin "2"
 		)
@@
 			)
 		)
+		(property "MPN" "GJM1555C1H2R7BB01D"
+			(at 0 0 0)
+			(effects
+				(font
+					(size 1.27 1.27)
+				)
+				(hide yes)
+			)
+		)
 		(pin "1"
 		)
@@
 			)
 		)
+		(property "MPN" "RC0402FR-07274KL"
+			(at 0 0 0)
+			(effects
+				(font
+					(size 1.27 1.27)
+				)
+				(hide yes)
+			)
+		)
 		(pin "2"
 		)
@@
 		(property "Package" "0402"
 			(at 117.856 65.532 90)
+			(effects
+				(font
+					(size 1.27 1.27)
+				)
+				(hide yes)
+			)
+		)
+		(property "MPN" "RC0402FR-070RL"
+			(at 0 0 0)
 			(effects
 				(font
@@
 			)
 		)
+		(property "MPN" "CL05C330JB5NNNC"
+			(at 0 0 0)
+			(effects
+				(font
+					(size 1.27 1.27)
+				)
+				(hide yes)
+			)
+		)
 		(pin "1"
 		)
@@
 			)
 		)
+		(property "MPN" "RC0402FR-0733RL"
+			(at 0 0 0)
+			(effects
+				(font
+					(size 1.27 1.27)
+				)
+				(hide yes)
+			)
+		)
 		(pin "1"
 		)
@@
 			)
 		)
+		(property "MPN" "INA240A3PW"
+			(at 0 0 0)
+			(effects
+				(font
+					(size 1.27 1.27)
+				)
+				(hide yes)
+			)
+		)
 		(pin "8"
 		)
@@
 			)
 		)
+		(property "MPN" "CL21A475KAQNNNE"
+			(at 0 0 0)
+			(effects
+				(font
+					(size 1.27 1.27)
+				)
+				(hide yes)
+			)
+		)
 		(pin "2"
 		)
@@
 			)
 		)
+		(property "MPN" "SIA400EDJ-T1-GE3"
+			(at 0 0 0)
+			(effects
+				(font
+					(size 1.27 1.27)
+				)
+				(hide yes)
+			)
+		)
 		(pin "1"
 		)
@@
 			(effects
 				(font
+					(size 1.27 1.27)
+				)
+				(hide yes)
+			)
+		)
+		(property "MPN" "RC0402FR-071KL"
+			(at 0 0 0)
+			(effects
+				(font
