File: hw/micro.kicad_sch (KiCad schematic)
At the start: 66 parts, among them J5 USB_C_Receptacle, J6 Conn_ST_STDC14, J7 TC2070, Q2 2N7002, SW2 MCU Reset, SW3 User1, SW4 SW_Nidec_CAS-120A1, U8 STSPIN32G4, U9 BNO055, Y1 25MHz

Commit message: More layout
Parts:
- removed R45, R46: 22.1k, Resistor_SMD:R_0402_1005Metric, symbol Device:R_Small
- renumbered R47 to R45
Connections:
- net 3V3: no longer C26.2, C27.2, C28.2
- net I2C_SCL: now also C28.2
- net USER_BTN_1: now also C27.2
- net nRST: now also C26.2
Other:
- note added: "Use internal pull-up resistor (~40k)"
- moved on the sheet: C26, C27, C28, R45, SW2, SW3, SW4, TP17, TP18, TP19

Commit message: layout 'finished' need to start double checking everything
Parts:
- added R43: 0Ω, Resistor_SMD:R_0402_1005Metric, symbol Device:R_Small
- added TP17: RGB_DIN_5V0, TestPoint:TestPoint_Pad_1.0x1.0mm, symbol Connector:TestPoint_Small
- renumbered NT1 to NT3, NT2 to NT4, NT3 to NT5, NT4 to NT6, NT5 to NT7, NT6 to NT8, R43 to R44, R44 to R45, R45 to R46, TP17 to TP18, TP18 to TP19, TP19 to TP20, TP20 to TP21
Connections:
- net DAC1_OUT: now also R43.1
- net RGB_DIN: now also NT3.1; no longer NT3.2
- net SPI3_MOSI: now also NT3.2; no longer NT3.1
- new net: R43.2, TP17.1
Changed lines of the file:
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@@
 	(wire
 		(pts
+			(xy 106.68 77.47) (xy 107.95 77.47)
+		)
+		(stroke
+			(width 0)
+			(type default)
+		)
+	)
+	(wire
+		(pts
 			(xy 227.33 148.59) (xy 227.33 156.21)
 		)
@@
 		(dnp no)
 		(fields_autoplaced yes)
-		(property "Reference" "NT2"
+		(property "Reference" "NT4"
 			(at 110.49 74.93 0)
 			(effects
@@
 			(project "bldc"
 				(path "/fdf9474f-66c9-4c2c-9436-f3125b555611/be5b0ca3-73b4-4a41-bf81-8399e62c0e5f"
-					(reference "NT2")
+					(reference "NT4")
 					(unit 1)
 				)
@@
 		(on_board yes)
 		(dnp no)
-		(property "Reference" "R45"
+		(property "Reference" "R46"
 			(at 157.48 110.49 0)
 			(effects
@@
 			(project "bldc"
 				(path "/fdf9474f-66c9-4c2c-9436-f3125b555611/be5b0ca3-73b4-4a41-bf81-8399e62c0e5f"
-					(reference "R45")
+					(reference "R46")
 					(unit 1)
 				)
@@
 	)
 	(symbol
+		(lib_id "Device:R_Small")
+		(at 110.49 77.47 270)
+		(unit 1)
+		(exclude_from_sim no)
+		(in_bom yes)
+		(on_board yes)
+		(dnp no)
+		(property "Reference" "R43"
+			(at 110.49 77.47 90)
+			(effects
+				(font
+					(size 1.016 1.016)
+				)
+			)
+		)
+		(property "Value" "0Ω"
+			(at 107.696 76.454 90)
+			(effects
+				(font
+					(size 1.27 1.27)
+				)
+			)
+		)
+		(property "Footprint" "Resistor_SMD:R_0402_1005Metric"
+			(at 110.49 77.47 0)
+			(effects
+				(font
+					(size 1.27 1.27)
+				)
+				(hide yes)
+			)
+		)
+		(property "Datasheet" "~"
+			(at 110.49 77.47 0)
+			(effects
+				(font
+					(size 1.27 1.27)
+				)
+				(hide yes)
+			)
+		)
+		(property "Description" "0Ω 0402"
+			(at 110.49 77.47 0)
+			(effects
+				(font
+					(size 1.27 1.27)
+				)
+				(hide yes)
+			)
+		)
+		(property "MFR.Part #" " RC0402FR-070RL"
+			(at 110.49 77.47 90)
+			(effects
+				(font
+					(size 1.27 1.27)
+				)
+				(hide yes)
+			)
+		)
+		(property "Package" "0402"
+			(at 106.934 75.438 90)
+			(effects
+				(font
+					(size 1.27 1.27)
+				)
+				(hide yes)
+			)
+		)
+		(pin "2"
+		)
+		(pin "1"
+		)
+		(instances
+			(project "bldc"
+				(path "/fdf9474f-66c9-4c2c-9436-f3125b555611/be5b0ca3-73b4-4a41-bf81-8399e62c0e5f"
+					(reference "R43")
+					(unit 1)
+				)
+			)
+		)
+	)
+	(symbol
 		(lib_id "Connector:TestPoint_Small")
 		(at 166.37 33.02 180)
@@
 		(dnp no)
 		(fields_autoplaced yes)
-		(property "Reference" "NT5"
+		(property "Reference" "NT7"
 			(at 213.36 135.89 0)
 			(effects
@@
 			(project "bldc"
 				(path "/fdf9474f-66c9-4c2c-9436-f3125b555611/be5b0ca3-73b4-4a41-bf81-8399e62c0e5f"
-					(reference "NT5")
+					(reference "NT7")
 					(unit 1)
 				)
@@
 		(on_board yes)
 		(dnp no)
-		(property "Reference" "TP17"
+		(property "Reference" "TP18"
 			(at 84.074 115.57 0)
 			(effects
@@
 			(project "bldc"
 				(path "/fdf9474f-66c9-4c2c-9436-f3125b555611/be5b0ca3-73b4-4a41-bf81-8399e62c0e5f"
-					(reference "TP17")
+					(reference "TP18")
 					(unit 1)
 				)
@@
 		(on_board yes)
 		(dnp no)
-		(property "Reference" "R44"
+		(property "Reference" "R45"
 			(at 46.99 99.06 90)
 			(effects
@@
 			(project "bldc"
 				(path "/fdf9474f-66c9-4c2c-9436-f3125b555611/be5b0ca3-73b4-4a41-bf81-8399e62c0e5f"
-					(reference "R44")
+					(reference "R45")
+					(unit 1)
+				)
+			)
+		)
+	)
+	(symbol
+		(lib_id "Connector:TestPoint_Small")
+		(at 106.68 77.47 0)
+		(unit 1)
+		(exclude_from_sim no)
+		(in_bom no)
+		(on_board yes)
+		(dnp no)
+		(property "Reference" "TP17"
+			(at 100.584 77.47 0)
+			(effects
+				(font
+					(size 1.27 1.27)
+				)
+				(justify left)
+			)
+		)
+		(property "Value" "RGB_DIN_5V0"
+			(at 107.95 78.7399 0)
+			(effects
+				(font
+					(size 1.27 1.27)
+				)
+				(justify left)
+				(hide yes)
+			)
+		)
+		(property "Footprint" "TestPoint:TestPoint_Pad_1.0x1.0mm"
+			(at 111.76 77.47 0)
+			(effects
+				(font
+					(size 1.27 1.27)
+				)
+				(hide yes)
+			)
+		)
+		(property "Datasheet" "~"
+			(at 111.76 77.47 0)
+			(effects
+				(font
+					(size 1.27 1.27)
+				)
+				(hide yes)
+			)
+		)
+		(property "Description" "test point"
+			(at 106.68 77.47 0)
+			(effects
+				(font
+					(size 1.27 1.27)
+				)
+				(hide yes)
+			)
+		)
+		(pin "1"
+		)
+		(instances
+			(project "bldc"
+				(path "/fdf9474f-66c9-4c2c-9436-f3125b555611/be5b0ca3-73b4-4a41-bf81-8399e62c0e5f"
+					(reference "TP17")
 					(unit 1)
 				)
@@
 		(on_board yes)
 		(dnp no)
-		(property "Reference" "TP20"
+		(property "Reference" "TP21"
 			(at 143.002 171.45 0)
 			(effects
@@
 			(project "bldc"
 				(path "/fdf9474f-66c9-4c2c-9436-f3125b555611/be5b0ca3-73b4-4a41-bf81-8399e62c0e5f"
-					(reference "TP20")
+					(reference "TP21")
 					(unit 1)
 				)
@@
 		(dnp no)
 		(fields_autoplaced yes)
-		(property "Reference" "NT4"
+		(property "Reference" "NT6"
 			(at 110.49 80.01 0)
 			(effects
@@
 			(project "bldc"
 				(path "/fdf9474f-66c9-4c2c-9436-f3125b555611/be5b0ca3-73b4-4a41-bf81-8399e62c0e5f"
-					(reference "NT4")
+					(reference "NT6")
 					(unit 1)
 				)
@@
 		(dnp no)
 		(fields_autoplaced yes)
-		(property "Reference" "NT3"
+		(property "Reference" "NT5"
 			(at 110.49 77.47 0)
 			(effects
@@
 			(project "bldc"
 				(path "/fdf9474f-66c9-4c2c-9436-f3125b555611/be5b0ca3-73b4-4a41-bf81-8399e62c0e5f"
-					(reference "NT3")
+					(reference "NT5")
 					(unit 1)
 				)
@@
 		(on_board yes)
 		(dnp no)
-		(property "Reference" "TP19"
+		(property "Reference" "TP20"
 			(at 184.404 115.57 0)
 			(effects
@@
 			(project "bldc"
 				(path "/fdf9474f-66c9-4c2c-9436-f3125b555611/be5b0ca3-73b4-4a41-bf81-8399e62c0e5f"
-					(reference "TP19")
+					(reference "TP20")
 					(unit 1)
 				)
@@
 		(on_board yes)
 		(dnp no)
-		(property "Reference" "TP18"
+		(property "Reference" "TP19"
 			(at 127.254 115.57 0)
 			(effects
@@
 			(project "bldc"
 				(path "/fdf9474f-66c9-4c2c-9436-f3125b555611/be5b0ca3-73b4-4a41-bf81-8399e62c0e5f"
-					(reference "TP18")
+					(reference "TP19")
 					(unit 1)
 				)
@@
 		(dnp no)
 		(fields_autoplaced yes)
-		(property "Reference" "NT6"
+		(property "Reference" "NT8"
 			(at 213.36 138.43 0)
 			(effects
@@
 			(project "bldc"
 				(path "/fdf9474f-66c9-4c2c-9436-f3125b555611/be5b0ca3-73b4-4a41-bf81-8399e62c0e5f"
-					(reference "NT6")
+					(reference "NT8")
 					(unit 1)
 				)
@@
 		(on_board yes)
 		(dnp yes)
-		(property "Reference" "R43"
+		(property "Reference" "R44"
 			(at 182.88 80.518 90)
 			(effects
@@
 			(project "bldc"
 				(path "/fdf9474f-66c9-4c2c-9436-f3125b555611/be5b0ca3-73b4-4a41-bf81-8399e62c0e5f"
-					(reference "R43")
+					(reference "R44")
 					(unit 1)
 				)
@@
 		(lib_id "Device:NetTie_2")
 		(at 175.26 44.45 0)
+		(mirror y)
 		(unit 1)
 		(exclude_from_sim no)
@@
 		(on_board yes)
 		(dnp no)
-		(fields_autoplaced yes)
-		(property "Reference" "NT1"
+		(property "Reference" "NT3"
 			(at 175.26 39.37 0)
 			(effects
@@
 			(project ""
 				(path "/fdf9474f-66c9-4c2c-9436-f3125b555611/be5b0ca3-73b4-4a41-bf81-8399e62c0e5f"
-					(reference "NT1")
+					(reference "NT3")
 					(unit 1)
 				)

Commit message: finalized / checked design
Parts:
- added NT10, NT12, NT9: NetTie_2, NetTie:NetTie-2_SMD_Pad0.5mm, symbol Device:NetTie_2
- C19, C21, C22, C25, C26, C27, C28, C29, C31, C32, C33, C35, C38: MPN (none) -> CL05B104KB54PNC
- C20, C30, C34, C37: MPN (none) -> CL21A475KAQNNNE
- C23, C24: MPN (none) -> CC0402KRNPO7BN100
- C36: MPN (none) -> CL21A106KAYNNNE
- D5, D6: MPN (none) -> 0603ESDA-05N
- D7: MPN (none) -> STPS1H100A
- J5: MPN (none) -> TYPE-C-31-M-12
- J6: MPN (none) -> FTSH-107-01-L-DV-K-A; Mfg. Part No. FTSH-107-01-L-DV-K-A -> FTSH-107-01-L-DV-K
- L2: MPN (none) -> MWSA0624S-150MT
- Q2: MPN (none) -> 2N7002
- R32, R33, R36, R46: MPN (none) -> RC0402FR-075K1L
- R34, R37, R38, R39, R40, R41, R42, R43, R44, R45: MPN (none) -> RC0402FR-070RL
- R35: MPN (none) -> RC0402FR-071KL
- SW2, SW3: MPN (none) -> B3FS-1052P
- SW4: MPN (none) -> CAS-120A1
- U8: MPN (none) -> STSPIN32G4
- U9: MPN (none) -> BNO055
- Y1: MPN (none) -> Q22FA12800569
Connections:
- net PHASE_U_VSENSE: now also NT10.1; no longer U8.16 (PA3)
- net PHASE_V_VSENSE: now also NT12.1; no longer U8.23 (PB0)
- net PHASE_W_VSENSE: now also NT9.1; no longer U8.14 (PA1)
- new net OPAMP1_VINP: NT10.2, U8.16 (PA3)
- new net OPAMP2_VINP: NT12.2, U8.23 (PB0)
- new net OPAMP3_VINP: NT9.2, U8.14 (PA1)
