File: hw/power-stage.kicad_sch (KiCad schematic)
At the start: 14 parts, among them U8 STSPIN32G4

Commit message: More layout
Parts:
- added C48: 4.7uF, Capacitor_SMD:C_0805_2012Metric, symbol Device:C_Small
- renumbered R48 to R46, R49 to R47, R50 to R48
Connections:
- net GND: now also C48.2
- net VBUS: now also C48.1
Changed lines of the file:
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@@
+	)
+	(junction
+		(at 168.91 38.1)
+		(diameter 0)
+		(color 0 0 0 0)
 	)
 	(junction
@@
 	)
 	(junction
+		(at 168.91 45.72)
+		(diameter 0)
+		(color 0 0 0 0)
+	)
+	(junction
 		(at 128.27 38.1)
 		(diameter 0)
@@
 	(wire
 		(pts
+			(xy 179.07 39.37) (xy 179.07 38.1)
+		)
+		(stroke
+			(width 0)
+			(type default)
+		)
+	)
+	(wire
+		(pts
 			(xy 95.25 102.87) (xy 107.95 102.87)
 		)
@@
 	(wire
 		(pts
+			(xy 179.07 44.45) (xy 179.07 45.72)
+		)
+		(stroke
+			(width 0)
+			(type default)
+		)
+	)
+	(wire
+		(pts
 			(xy 133.35 92.71) (xy 142.24 92.71)
 		)
@@
 	(wire
 		(pts
+			(xy 168.91 45.72) (xy 179.07 45.72)
+		)
+		(stroke
+			(width 0)
+			(type default)
+		)
+	)
+	(wire
+		(pts
 			(xy 62.23 92.71) (xy 72.39 92.71)
+		)
+		(stroke
+			(width 0)
+			(type default)
+		)
+	)
+	(wire
+		(pts
+			(xy 179.07 38.1) (xy 168.91 38.1)
 		)
 		(stroke
@@
 		(dnp no)
 		(fields_autoplaced yes)
-		(property "Reference" "#PWR090"
+		(property "Reference" "#PWR088"
 			(at 68.58 120.65 0)
 			(effects
@@
 			(project "bldc"
 				(path "/fdf9474f-66c9-4c2c-9436-f3125b555611/066314e2-1f8c-41a2-8da1-0e67cde6d8c9"
-					(reference "#PWR090")
+					(reference "#PWR088")
+					(unit 1)
+				)
+			)
+		)
+	)
+	(symbol
+		(lib_id "Device:C_Small")
+		(at 179.07 41.91 0)
+		(unit 1)
+		(exclude_from_sim no)
+		(in_bom yes)
+		(on_board yes)
+		(dnp no)
+		(fields_autoplaced yes)
+		(property "Reference" "C48"
+			(at 181.61 40.6462 0)
+			(effects
+				(font
+					(size 1.27 1.27)
+				)
+				(justify left)
+			)
+		)
+		(property "Value" "4.7uF"
+			(at 181.61 43.1862 0)
+			(effects
+				(font
+					(size 1.27 1.27)
+				)
+				(justify left)
+			)
+		)
+		(property "Footprint" "Capacitor_SMD:C_0805_2012Metric"
+			(at 179.07 41.91 0)
+			(effects
+				(font
+					(size 1.27 1.27)
+				)
+				(hide yes)
+			)
+		)
+		(property "Datasheet" "~"
+			(at 179.07 41.91 0)
+			(effects
+				(font
+					(size 1.27 1.27)
+				)
+				(hide yes)
+			)
+		)
+		(property "Description" "Unpolarized capacitor, small symbol"
+			(at 179.07 41.91 0)
+			(effects
+				(font
+					(size 1.27 1.27)
+				)
+				(hide yes)
+			)
+		)
+		(property "Mfg. Part No." "CL21A475KAQNNNE"
+			(at 179.07 41.91 0)
+			(effects
+				(font
+					(size 1.27 1.27)
+				)
+				(hide yes)
+			)
+		)
+		(property "Voltage" "25V"
+			(at 179.07 41.91 0)
+			(effects
+				(font
+					(size 1.27 1.27)
+				)
+				(hide yes)
+			)
+		)
+		(pin "2"
+		)
+		(pin "1"
+		)
+		(instances
+			(project "bldc"
+				(path "/fdf9474f-66c9-4c2c-9436-f3125b555611/066314e2-1f8c-41a2-8da1-0e67cde6d8c9"
+					(reference "C48")
 					(unit 1)
 				)
@@
 		(on_board yes)
 		(dnp no)
-		(property "Reference" "#PWR086"
+		(property "Reference" "#PWR084"
 			(at 68.58 78.74 0)
 			(effects
@@
 			(project "bldc"
 				(path "/fdf9474f-66c9-4c2c-9436-f3125b555611/066314e2-1f8c-41a2-8da1-0e67cde6d8c9"
-					(reference "#PWR086")
+					(reference "#PWR084")
 					(unit 1)
 				)
@@
 		(on_board yes)
 		(dnp no)
-		(property "Reference" "R48"
+		(property "Reference" "R46"
 			(at 53.34 87.884 0)
 			(effects
@@
 			(project "bldc"
 				(path "/fdf9474f-66c9-4c2c-9436-f3125b555611/066314e2-1f8c-41a2-8da1-0e67cde6d8c9"
-					(reference "R48")
+					(reference "R46")
 					(unit 1)
 				)
@@
 		(on_board yes)
 		(dnp no)
-		(property "Reference" "#PWR084"
+		(property "Reference" "#PWR082"
 			(at 87.63 40.64 0)
 			(effects
@@
 			(project "bldc"
 				(path "/fdf9474f-66c9-4c2c-9436-f3125b555611/066314e2-1f8c-41a2-8da1-0e67cde6d8c9"
-					(reference "#PWR084")
+					(reference "#PWR082")
 					(unit 1)
 				)
@@
 		(on_board yes)
 		(dnp no)
-		(property "Reference" "R49"
+		(property "Reference" "R47"
 			(at 51.562 94.996 0)
 			(effects
@@
 			(project "bldc"
 				(path "/fdf9474f-66c9-4c2c-9436-f3125b555611/066314e2-1f8c-41a2-8da1-0e67cde6d8c9"
-					(reference "R49")
+					(reference "R47")
 					(unit 1)
 				)
@@
 		(on_board yes)
 		(dnp no)
-		(property "Reference" "#PWR087"
+		(property "Reference" "#PWR085"
 			(at 58.42 87.63 0)
 			(effects
@@
 			(project "bldc"
 				(path "/fdf9474f-66c9-4c2c-9436-f3125b555611/066314e2-1f8c-41a2-8da1-0e67cde6d8c9"
-					(reference "#PWR087")
+					(reference "#PWR085")
 					(unit 1)
 				)
@@
 		(dnp no)
 		(fields_autoplaced yes)
-		(property "Reference" "#PWR085"
+		(property "Reference" "#PWR083"
 			(at 87.63 54.61 0)
 			(effects
@@
 			(project "bldc"
 				(path "/fdf9474f-66c9-4c2c-9436-f3125b555611/066314e2-1f8c-41a2-8da1-0e67cde6d8c9"
-					(reference "#PWR085")
+					(reference "#PWR083")
 					(unit 1)
 				)
@@
 		(on_board yes)
 		(dnp no)
-		(property "Reference" "#PWR088"
+		(property "Reference" "#PWR086"
 			(at 68.58 87.63 0)
 			(effects
@@
 			(project "bldc"
 				(path "/fdf9474f-66c9-4c2c-9436-f3125b555611/066314e2-1f8c-41a2-8da1-0e67cde6d8c9"
-					(reference "#PWR088")
+					(reference "#PWR086")
 					(unit 1)
 				)
@@
 		(on_board yes)
 		(dnp no)
-		(property "Reference" "R50"
+		(property "Reference" "R48"
 			(at 59.944 95.25 0)
 			(effects
@@
 			(project "bldc"
 				(path "/fdf9474f-66c9-4c2c-9436-f3125b555611/066314e2-1f8c-41a2-8da1-0e67cde6d8c9"
-					(reference "R50")
+					(reference "R48")
 					(unit 1)
 				)
@@
 					(unit 3)
 				)
-				(path "/fdf9474f-66c9-4c2c-9436-f3125b555611/be5b0ca3-73b4-4a41-bf81-8399e62c0e5f"
-					(reference "U?")
-					(unit 3)
-				)
 			)
 		)
@@
 		(dnp no)
 		(fields_autoplaced yes)
-		(property "Reference" "#PWR089"
+		(property "Reference" "#PWR087"
 			(at 57.15 107.95 0)
 			(effects
@@
 			(project "bldc"
 				(path "/fdf9474f-66c9-4c2c-9436-f3125b555611/066314e2-1f8c-41a2-8da1-0e67cde6d8c9"
-					(reference "#PWR089")
+					(reference "#PWR087")
 					(unit 1)
 				)

Commit message: layout 'finished' need to start double checking everything
Parts:
- renumbered R46 to R47, R47 to R48, R48 to R49, TP21 to TP22
Changed lines of the file:
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@@
-	(wire
-		(pts
-			(xy 171.45 119.38) (xy 175.26 119.38)
-		)
-		(stroke
-			(width 0)
-			(type default)
-		)
-	)
-	(wire
-		(pts
-			(xy 171.45 99.06) (xy 175.26 99.06)
-		)
-		(stroke
-			(width 0)
-			(type default)
-		)
-	)
 	(wire
 		(pts
@@
 	(wire
 		(pts
+			(xy 175.26 116.84) (xy 171.45 116.84)
+		)
+		(stroke
+			(width 0)
+			(type default)
+		)
+	)
+	(wire
+		(pts
 			(xy 168.91 38.1) (xy 158.75 38.1)
 		)
@@
 	(wire
 		(pts
+			(xy 175.26 96.52) (xy 171.45 96.52)
+		)
+		(stroke
+			(width 0)
+			(type default)
+		)
+	)
+	(wire
+		(pts
 			(xy 133.35 115.57) (xy 142.24 115.57)
 		)
@@
 	(wire
 		(pts
-			(xy 171.45 96.52) (xy 175.26 96.52)
-		)
-		(stroke
-			(width 0)
-			(type default)
-		)
-	)
-	(wire
-		(pts
 			(xy 138.43 39.37) (xy 138.43 38.1)
 		)
@@
 	(wire
 		(pts
-			(xy 171.45 116.84) (xy 175.26 116.84)
+			(xy 175.26 119.38) (xy 171.45 119.38)
 		)
 		(stroke
@@
 		(pts
 			(xy 87.63 44.45) (xy 87.63 45.72)
+		)
+		(stroke
+			(width 0)
+			(type default)
+		)
+	)
+	(wire
+		(pts
+			(xy 175.26 99.06) (xy 171.45 99.06)
 		)
 		(stroke
@@
 	(hierarchical_label "V_ISENSE"
 		(shape output)
-		(at 175.26 99.06 0)
+		(at 175.26 96.52 0)
 		(effects
 			(font
@@
 	(hierarchical_label "W_VSENSE"
 		(shape output)
-		(at 175.26 116.84 0)
+		(at 175.26 119.38 0)
 		(effects
 			(font
@@
 	(hierarchical_label "V_VSENSE"
 		(shape output)
-		(at 175.26 96.52 0)
+		(at 175.26 99.06 0)
 		(effects
 			(font
@@
 	(hierarchical_label "W_ISENSE"
 		(shape output)
-		(at 175.26 119.38 0)
+		(at 175.26 116.84 0)
 		(effects
 			(font
@@
 		(on_board yes)
 		(dnp no)
-		(property "Reference" "R46"
+		(property "Reference" "R47"
 			(at 53.34 87.884 0)
 			(effects
@@
 			(project "bldc"
 				(path "/fdf9474f-66c9-4c2c-9436-f3125b555611/066314e2-1f8c-41a2-8da1-0e67cde6d8c9"
-					(reference "R46")
+					(reference "R47")
 					(unit 1)
 				)
@@
 		(on_board yes)
 		(dnp no)
-		(property "Reference" "TP21"
+		(property "Reference" "TP22"
 			(at 60.452 90.932 0)
 			(effects
@@
 			(project "bldc"
 				(path "/fdf9474f-66c9-4c2c-9436-f3125b555611/066314e2-1f8c-41a2-8da1-0e67cde6d8c9"
-					(reference "TP21")
+					(reference "TP22")
 					(unit 1)
 				)
@@
 		(on_board yes)
 		(dnp no)
-		(property "Reference" "R47"
+		(property "Reference" "R48"
 			(at 51.562 94.996 0)
 			(effects
@@
 			(project "bldc"
 				(path "/fdf9474f-66c9-4c2c-9436-f3125b555611/066314e2-1f8c-41a2-8da1-0e67cde6d8c9"
-					(reference "R47")
+					(reference "R48")
 					(unit 1)
 				)
@@
 		(on_board yes)
 		(dnp no)
-		(property "Reference" "R48"
+		(property "Reference" "R49"
 			(at 59.944 95.25 0)
 			(effects
@@
 			(project "bldc"
 				(path "/fdf9474f-66c9-4c2c-9436-f3125b555611/066314e2-1f8c-41a2-8da1-0e67cde6d8c9"
-					(reference "R48")
+					(reference "R49")
 					(unit 1)
 				)

Commit message: finalized / checked design
Parts:
- C39, C40, C41, C42, C43, C44, C45, C46, C47, C48: MPN (none) -> CL21A475KAQNNNE
- R47: MPN (none) -> RC0402FR-0722K1L
- R48, R49: MPN (none) -> RC0402FR-075K1L
- U8: MPN (none) -> STSPIN32G4
Changed lines of the file:
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@@
+			)
+		)
+		(property "MPN" "CL21A475KAQNNNE"
+			(at 0 0 0)
+			(effects
+				(font
+					(size 1.27 1.27)
+				)
+				(hide yes)
 			)
 		)
@@
 			)
 		)
+		(property "MPN" "CL21A475KAQNNNE"
+			(at 0 0 0)
+			(effects
+				(font
+					(size 1.27 1.27)
+				)
+				(hide yes)
+			)
+		)
 		(pin "2"
 		)
@@
 			)
 		)
+		(property "MPN" "CL21A475KAQNNNE"
+			(at 0 0 0)
+			(effects
+				(font
+					(size 1.27 1.27)
+				)
+				(hide yes)
+			)
+		)
 		(pin "2"
 		)
@@
 			)
 		)
+		(property "MPN" "CL21A475KAQNNNE"
+			(at 0 0 0)
+			(effects
+				(font
+					(size 1.27 1.27)
+				)
+				(hide yes)
+			)
+		)
 		(pin "2"
 		)
@@
 			)
 		)
+		(property "MPN" "CL21A475KAQNNNE"
+			(at 0 0 0)
+			(effects
+				(font
+					(size 1.27 1.27)
+				)
+				(hide yes)
+			)
+		)
 		(pin "2"
 		)
@@
 		(property "Mfg. Part No." "RC0402FR-0722K1L"
 			(at 58.42 88.9 0)
+			(effects
+				(font
+					(size 1.27 1.27)
+				)
+				(hide yes)
+			)
+		)
+		(property "MPN" "RC0402FR-0722K1L"
+			(at 0 0 0)
 			(effects
 				(font
@@
 			)
 		)
+		(property "MPN" "CL21A475KAQNNNE"
+			(at 0 0 0)
+			(effects
+				(font
+					(size 1.27 1.27)
+				)
+				(hide yes)
+			)
+		)
 		(pin "2"
 		)
@@
 			)
 		)
+		(property "MPN" "CL21A475KAQNNNE"
+			(at 0 0 0)
+			(effects
+				(font
+					(size 1.27 1.27)
+				)
+				(hide yes)
+			)
+		)
 		(pin "2"
 		)
@@
 		(property "Mfg. Part No." "RC0402FR-075K1L"
 			(at 55.88 96.52 0)
+			(effects
+				(font
+					(size 1.27 1.27)
+				)
+				(hide yes)
+			)
+		)
+		(property "MPN" "RC0402FR-075K1L"
+			(at 0 0 0)
 			(effects
 				(font
@@
 			)
 		)
+		(property "MPN" "CL21A475KAQNNNE"
+			(at 0 0 0)
+			(effects
+				(font
+					(size 1.27 1.27)
+				)
+				(hide yes)
+			)
+		)
 		(pin "2"
 		)
@@
 			)
 		)
+		(property "MPN" "RC0402FR-075K1L"
+			(at 0 0 0)
+			(effects
+				(font
+					(size 1.27 1.27)
+				)
+				(hide yes)
+			)
+		)
 		(pin "1"
 		)
@@
 			)
 		)
+		(property "MPN" "CL21A475KAQNNNE"
+			(at 0 0 0)
+			(effects
+				(font
+					(size 1.27 1.27)
+				)
+				(hide yes)
+			)
+		)
 		(pin "2"
 		)
@@
 			)
 		)
+		(property "MPN" "CL21A475KAQNNNE"
+			(at 0 0 0)
+			(effects
+				(font
+					(size 1.27 1.27)
+				)
+				(hide yes)
+			)
+		)
 		(pin "2"
 		)
@@
 			(effects
 				(font
+					(size 1.27 1.27)
+				)
+				(hide yes)
+			)
+		)
+		(property "MPN" "STSPIN32G4"
+			(at 0 0 0)
+			(effects
+				(font
