File: hw/usb-pd.kicad_sch (KiCad schematic)
At the start: 74 parts, among them J4 USB_C_Receptacle, Q1 2N7002K, SW1 SW_Nidec_CAS-120A1, U1 CSD25402Q3A, U2 CSD25402Q3A, U3 INA180A2, U4 CYPD3177-24LQ, U5 LMR50410, U6 LD1117S33TR_SOT223, U7 TPS2116DRL

Commit message: More layout
Parts:
- added NT10, NT11: NetTie_2, NetTie:NetTie-2_SMD_Pad0.5mm, symbol Device:NetTie_2
- renumbered R29 to R28, R28 to R29, R31 to R30, R30 to R31
Connections:
- net 3V3: now also R28.1; no longer D3.2 (A)
- net 5V0_BUCK: now also R22.1; no longer D2.2 (A)
- net GND: now also D2.1 (K), D3.1 (K), D4.1 (K); no longer R22.2, R28.2, R30.2
- net MCU_USB_VBUS: now also R30.1; no longer D4.2 (A)
- net VBUS: now also NT11.2; no longer U3.4 (-)
- net VBUS_ISENSE_HI: now also NT10.1; no longer C4.1, R1.1, U2.1 (D), U2.2 (D), U2.3 (D), U4.11 (VDC_OUT)
- net VBUS_FET_SW: now reaches R5.1, R6.1, U1.5 (S), U2.5 (S)
- net VBUS_FET_GATE: now reaches C3.1, C4.2, R10.2, R3.2, R4.2, R5.2, R6.2, R9.2, U1.4 (G), U2.4 (G)
- new net: D2.2 (A), R22.2
- new net: D4.2 (A), R30.2
- new net: D3.2 (A), R28.2
- new net VBUS_ISENSE_LOW: NT11.1, U3.4 (-)
- new net VDC_OUT: C4.1, NT10.2, R1.1, U2.1 (D), U2.2 (D), U2.3 (D), U4.11 (VDC_OUT)
Other:
- moved on the sheet: C13, D2, D3, D4, R22, R28, R30, TP6

Commit message: layout 'finished' need to start double checking everything
Parts:
- TP6: value 5V0_VSENSE -> VBUS
- TP8: value 5V0_VSENSE -> 5V0
- TP9: value 5V0_VSENSE -> 3V3
- renumbered NT10 to NT1, NT11 to NT2
Other:
- moved on the sheet: D1
Changed lines of the file:
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@@
 			)
 		)
-		(property "Value" "5V0_VSENSE"
+		(property "Value" "VBUS"
 			(at 25.4 114.2999 0)
 			(effects
@@
 			)
 		)
-		(property "Value" "5V0_VSENSE"
+		(property "Value" "3V3"
 			(at 140.97 160.0199 0)
 			(effects
@@
 		(dnp no)
 		(fields_autoplaced yes)
-		(property "Reference" "NT10"
+		(property "Reference" "NT1"
 			(at 180.34 31.75 0)
 			(effects
@@
 			(project "bldc"
 				(path "/fdf9474f-66c9-4c2c-9436-f3125b555611/ea8b7c77-38a2-4626-ae83-899cfe040239"
-					(reference "NT10")
+					(reference "NT1")
 					(unit 1)
 				)
@@
 			)
 		)
-		(property "Value" "5V0_VSENSE"
+		(property "Value" "5V0"
 			(at 96.52 160.0199 0)
 			(effects
@@
 		(dnp no)
 		(fields_autoplaced yes)
-		(property "Reference" "NT11"
+		(property "Reference" "NT2"
 			(at 200.66 31.75 0)
 			(effects
@@
 			(project "bldc"
 				(path "/fdf9474f-66c9-4c2c-9436-f3125b555611/ea8b7c77-38a2-4626-ae83-899cfe040239"
-					(reference "NT11")
+					(reference "NT2")
 					(unit 1)
 				)
@@
 		(on_board yes)
 		(dnp no)
-		(fields_autoplaced yes)
 		(property "Reference" "U3"
 			(at 256.54 58.3498 0)
@@
 		(lib_id "Device:C_Small")
 		(at 170.18 31.75 0)
+		(mirror y)
 		(unit 1)
 		(exclude_from_sim no)
@@
 		(on_board yes)
 		(dnp no)
-		(fields_autoplaced yes)
 		(property "Reference" "C4"
-			(at 172.72 30.4862 0)
+			(at 167.64 30.4862 0)
 			(effects
 				(font
@@
 		)
 		(property "Value" "4.7uF"
-			(at 172.72 33.0262 0)
+			(at 167.64 33.0262 0)
 			(effects
 				(font
@@
 	(symbol
 		(lib_id "Device:LED_Small")
-		(at 220.98 85.09 90)
+		(at 220.98 85.09 270)
+		(mirror x)
 		(unit 1)
 		(exclude_from_sim no)
@@
 		(on_board yes)
 		(dnp no)
-		(fields_autoplaced yes)
 		(property "Reference" "D1"
-			(at 223.52 83.7564 90)
+			(at 218.44 83.7564 90)
 			(effects
 				(font
@@
 		)
 		(property "Value" "Red"
-			(at 223.52 86.2964 90)
+			(at 218.44 86.2964 90)
 			(effects
 				(font

Commit message: finalized / checked design
Parts:
- removed R14, R15: 2.4k, Resistor_SMD:R_0402_1005Metric, symbol Device:R_Small
- C1, C3, C4, C7, C8: MPN (none) -> CL21A475KAQNNNE
- C10, C11, C12, C15, C16, C17, C2, C5, C6, C9: MPN (none) -> CL05B104KB54PNC
- C13: MPN (none) -> CL21B225KAFNNNE
- C14: MPN (none) -> CL21A226MAQNNNE
- C18: MPN (none) -> CL21A106KAYNNNE
- D1: MPN (none) -> LTST-C191KRKT
- D2, D3, D4: MPN (none) -> LTST-C193TGKT-5A
- J4: MPN (none) -> TYPE-C-31-M-12
- L1: MPN (none) -> MWSA0624S-150MT
- Q1: MPN (none) -> 2N7002K-7
- R1: MPN (none) -> HoYH1206-1W-12mR-1%
- R10, R11, R13, R16, R17, R18, R19, R7, R8, R9: MPN (none) -> RC0402FR-072K4L
- R12, R24, R25, R26, R27, R29, R31: MPN (none) -> RC0402FR-075K1L
- R2: MPN (none) -> RC0402FR-076K8L
- R20, R23, R3, R4: MPN (none) -> RC0402FR-0722K1L
- R21, R5, R6: MPN (none) -> RC0402FR-0788K7L
- R22, R28, R30: MPN (none) -> RC0402FR-07470RL
- SW1: MPN (none) -> CAS-120A1
- U1, U2: MPN (none) -> CSD25402Q3A
- U3: MPN (none) -> INA180A2IDBVR
- U4: MPN (none) -> CYPD3177-24LQXQ
- U5: MPN (none) -> LMR50410XDDCR
- U6: MPN (none) -> LD1117S33TR
- U7: MPN (none) -> TPS2116DRLR
