File: hw/stm32h7/pcs_bldc_h7.kicad_pcb (KiCad board)
At the start: 2 copper layers, 35.5 x 69.9 mm, 120 parts, among them J1 USB_C_Receptacle, J10 miniPCIe, J11 Bus_PCI_Express_Mini, J12 2-1445100-3, J13 Encoder, J2 TC2030, J3 2-1445100-3, J4 Encoder, J5 436500212, J6 RJ45_Hanrun_HR911105A_Horizon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, J7 RJ45_Hanrun_HR911105A_Horizon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, J8 FDCAN2, J9 FDCAN1, SW1 MCU Reset, SW2 MCU Reset, U1 USBLC6-2P6, U2 STM32H743VIHx, U3 DRV8316C, U4 LMR50410, U5 INA241A3xDDF, U6 TPS2116DRL, U7 TLV75733PDRV, U8 TLV75733PDRV, U9 DRV8316C

Commit message: WIP: H7 dual-axis encoder ports, VSENSE, LED swap, TPS2553/ESD on J4
- driver sheet: respaced; DRV8316C 3x-PWM pinout; J4 encoder port with
  100R series, 2.2k/5.1k pull-ups, TPD4E05U06 ESD array, TPS2553 current
  limited 5V switch (ENC_EN/ENC_SW_nFLT); phase VSENSE dividers
  (100k/8.2k, 8.2p/100p compensated); R55/R58/R62 footprint -> R_0201
- root sheet: second driver instance (driver2) for the dual-axis plan
- micro sheet: D1/D2 -> WS2812B-2020-V6 (3.3V logic), 5V0 feed
- power sheet: drop 3V3_VSENSE_AI (VREFINT instead), LMR50410 cleanup
- stm32h7.ioc: TIM1/TIM8 PWM, SPI2/SPI3/SPI4, TIM4 encoder, FDCAN1/2,
  QUADSPI bank 2
- datasheets: WS2812B-2020-V6, SK6805-EC15, TPS2553
Parts:
- added C15: 0.1uF, Capacitor_SMD:C_0201_0603Metric, F.Cu at (191.6, 143.4)
- added C18: 0.1uF, Capacitor_SMD:C_0201_0603Metric, F.Cu at (191.6, 145.1)
- added R11: 100R, Resistor_SMD:R_0201_0603Metric, F.Cu at (181.1, 92.1)
- added R12: 100R, Resistor_SMD:R_0201_0603Metric, F.Cu at (181.1, 93.8)
- added R13: 100R, Resistor_SMD:R_0201_0603Metric, F.Cu at (181.1, 95.6)
- added R14: 100R, Resistor_SMD:R_0201_0603Metric, F.Cu at (181.1, 97.3)
- added R15: 2.2k, Resistor_SMD:R_0201_0603Metric, F.Cu at (181.1, 99.1)
- added R16: 2.2k, Resistor_SMD:R_0201_0603Metric, F.Cu at (181.1, 100.8)
- added R17: 2.2k, Resistor_SMD:R_0201_0603Metric, F.Cu at (181.1, 102.6)
- added R3: 0R, Resistor_SMD:R_0201_0603Metric, F.Cu at (191.6, 146.9)
- added R36: 100R, Resistor_SMD:R_0201_0603Metric, F.Cu at (181.1, 77.8)
- added R37: 100R, Resistor_SMD:R_0201_0603Metric, F.Cu at (181.1, 79.6)
- added R38: 100R, Resistor_SMD:R_0201_0603Metric, F.Cu at (181.1, 81.3)
- added R39: 100R, Resistor_SMD:R_0201_0603Metric, F.Cu at (181.1, 83.1)
- added R40: 2.2k, Resistor_SMD:R_0201_0603Metric, F.Cu at (181.1, 84.8)
- added R41: 2.2k, Resistor_SMD:R_0201_0603Metric, F.Cu at (181.1, 86.6)
- added R42: 2.2k, Resistor_SMD:R_0201_0603Metric, F.Cu at (181.1, 88.3)
- added TP3: 5V0_VSENSE, TestPoint:TestPoint_Pad_1.0x1.0mm, F.Cu at (191.9, 149.3)
- added U11: TPD4E05U06DQA, Package_SON:USON-10_2.5x1.0mm_P0.5mm, F.Cu at (183.8, 87.1)
- added U4: TPD4E05U06DQA, Package_SON:USON-10_2.5x1.0mm_P0.5mm, F.Cu at (183.8, 101.3)
- D1, D2: value SK6805 -> WS2812B-2020; footprint LED_SMD:LED_SK6805_PLCC4_2.4x2.7mm_P1.3mm -> pcs_lib:LED_WS2812B-2020_PLCC4_2.0x2.0mm
- J13, J4: footprint Connector_Molex:Molex_PicoBlade_53261-0571_1x05-1MP_P1.25mm_Horizontal -> Connector_Molex:Molex_PicoBlade_53261-0671_1x06-1MP_P1.25mm_Horizontal
- moved D1 73.5 mm to (192.5, 137.2)
- moved D2 70.7 mm to (192.5, 140.7)
- moved U2 8.03 mm to (156.2, 129.5)
- renumbered C15 to C16, C16 to C17, C17 to C19, C18 to C20, C19 to C21, C20 to C22, C21 to C23, C22 to C24, C23 to C25, C24 to C26, C25 to C27, C26 to C28, C27 to C29, C28 to C30, C29 to C31, C30 to C32, C31 to C33, C32 to C34, C33 to C35, C34 to C36, C35 to C37, C36 to C38, C37 to C39, C38 to C40, C39 to C41, C40 to C42, C41 to C43, C42 to C44, C43 to C45, C44 to C46, C45 to C47, C46 to C48, C47 to C49, C48 to C50, C49 to C51, C50 to C52, C51 to C53, C52 to C54, C53 to C55, C54 to C56, R9 to R10, R10 to R18, R11 to R19, R12 to R20, R13 to R21, R14 to R22, R15 to R23, R16 to R24, R17 to R25, R18 to R26, R19 to R27, R20 to R28, R21 to R29, R22 to R30, R23 to R31, R24 to R32, R25 to R33, R26 to R34, R27 to R35, R3 to R4, R4 to R5, R5 to R6, R6 to R7, R7 to R8, R8 to R9, TP9 to TP10, TP3 to TP4, TP4 to TP5, TP5 to TP6, TP6 to TP7, TP7 to TP8, TP8 to TP9, U9 to U10, U4 to U5, U5 to U6, U6 to U7, U7 to U8, U8 to U9
Connections:
- D1 pad 1: unconnected-(D1-DOUT-Pad1) -> Net-(D1-DOUT)
- D1 pad 2: unconnected-(D1-VSS-Pad2) -> GND
- D1 pad 3: unconnected-(D1-DIN-Pad3) -> Net-(D1-DIN)
- D1 pad 4: unconnected-(D1-VDD-Pad4) -> 5V0
- D2 pad 1: unconnected-(D2-DOUT-Pad1) -> Net-(D2-DOUT)
- D2 pad 2: unconnected-(D2-VSS-Pad2) -> GND
- D2 pad 3: unconnected-(D2-DIN-Pad3) -> Net-(D1-DOUT)
- D2 pad 4: unconnected-(D2-VDD-Pad4) -> 5V0
- J13 pad 1: unconnected-(J13-Pin_1-Pad1) -> Net-(J13-Pin_1)
- J13 pad 2: unconnected-(J13-Pin_2-Pad2) -> Net-(J13-Pin_2)
- J13 pad 3: unconnected-(J13-Pin_3-Pad3) -> Net-(J13-Pin_3)
- J13 pad 4: unconnected-(J13-Pin_4-Pad4) -> Net-(J13-Pin_4)
- J13 pad 5: unconnected-(J13-Pin_5-Pad5) -> 5V0
- J4 pad 1: unconnected-(J4-Pin_1-Pad1) -> Net-(J4-Pin_1)
- J4 pad 2: unconnected-(J4-Pin_2-Pad2) -> Net-(J4-Pin_2)
- J4 pad 3: unconnected-(J4-Pin_3-Pad3) -> Net-(J4-Pin_3)
- J4 pad 4: unconnected-(J4-Pin_4-Pad4) -> Net-(J4-Pin_4)
- J4 pad 5: unconnected-(J4-Pin_5-Pad5) -> 5V0
- U2 pad A10: unconnected-(U2-PA13-PadA10) -> /micro/SWDIO
- U2 pad A7: unconnected-(U2-PB3-PadA7) -> /micro/SWO
- U2 pad A9: unconnected-(U2-PA14-PadA9) -> /micro/SWCLK
