File: hw/stm32h7/pcs_bldc_h7.kicad_pcb (KiCad board)
At the start: 2 copper layers, 35.5 x 69.9 mm, 140 parts, among them J1 USB_C_Receptacle, J10 miniPCIe, J11 Bus_PCI_Express_Mini, J12 2-1445100-3, J13 Encoder, J2 TC2030, J3 2-1445100-3, J4 Encoder, J5 436500212, J6 RJ45_Hanrun_HR911105A_Horizon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, J7 RJ45_Hanrun_HR911105A_Horizon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, J8 FDCAN2, J9 FDCAN1, SW1 MCU Reset, SW2 MCU Reset, U1 USBLC6-2P6, U10 DRV8316C, U11 TPD4E05U06DQA, U2 STM32H743VIHx, U3 DRV8316C, U4 TPD4E05U06DQA, U5 LMR50410, U6 INA241A3xDDF, U7 TPS2116DRL, U8 TLV75733PDRV, U9 TLV75733PDRV

Commit message: WIP: H7 schematic and PCB layout progress
Parts:
- removed the C46 at (211.0, 44.4)
- removed the C47 at (198.1, 58.2)
- removed the C48 at (198.1, 61.2)
- removed the C49 at (211.0, 46.3)
- removed the C50 at (211.0, 48.3)
- removed the C51 at (211.0, 50.3)
- removed the C52 at (211.0, 52.2)
- removed the C54 at (208.3, 44.0)
- removed the C55 at (208.3, 45.8)
- removed the C56 at (208.3, 47.5)
- removed the J12 at (161.3, 95.7)
- removed the J13 at (161.3, 90.2)
- removed the R29 at (120.2, 96.9)
- removed the R30 at (120.2, 98.9)
- removed the R31 at (201.8, 57.7)
- removed the R32 at (208.3, 49.3)
- removed the R33 at (208.3, 51.0)
- removed the R34 at (208.3, 52.8)
- removed the R35 at (208.3, 54.5)
- removed the R36 at (181.1, 77.8)
- removed the R37 at (181.1, 79.6)
- removed the R38 at (181.1, 81.3)
- removed the R39 at (181.1, 83.1)
- removed the TP2 at (196.5, 116.8)
- removed the U10 at (157.5, 109.2)
- added C19: 0.1uF, Capacitor_SMD:C_0201_0603Metric, F.Cu at (135.6, 95.5)
- added C20: 0.1uF, Capacitor_SMD:C_0201_0603Metric, F.Cu at (169.2, 95.0)
- added C23: 0.1uF, Capacitor_SMD:C_0201_0603Metric, F.Cu at (135.6, 98.0)
- added C24: 0.1uF, Capacitor_SMD:C_0201_0603Metric, F.Cu at (169.2, 97.5)
- added C3: 8pF, Capacitor_SMD:C_0201_0603Metric, B.Cu at (159.8, 138.4)
- added C38: 0.1uF, Capacitor_SMD:C_0201_0603Metric, B.Cu at (167.6, 117.1)
- added C39: 8.2pF, Capacitor_SMD:C_0201_0603Metric, B.Cu at (148.3, 99.3)
- added C40: 100pF, Capacitor_SMD:C_0201_0603Metric, B.Cu at (150.1, 99.3)
- added C42: 8.2pF, Capacitor_SMD:C_0201_0603Metric, B.Cu at (148.3, 101.3)
- added C43: 100pF, Capacitor_SMD:C_0201_0603Metric, B.Cu at (150.1, 101.3)
- added C5: 8pF, Capacitor_SMD:C_0201_0603Metric, B.Cu at (160.8, 138.4)
- added C58: 0.1uF, Capacitor_SMD:C_0201_0603Metric, B.Cu at (166.1, 124.7)
- added C59: 22uF, Capacitor_SMD:C_0603_1608Metric, F.Cu at (195.3, 126.8)
- added C60: 47nF, Capacitor_SMD:C_0402_1005Metric, F.Cu at (191.9, 118.6)
- added C61: 1uF, Capacitor_SMD:C_0402_1005Metric, F.Cu at (191.9, 120.5)
- added C62: 10uF, Capacitor_SMD:C_0805_2012Metric, F.Cu at (182.9, 123.9)
- added C63: 10uF, Capacitor_SMD:C_0805_2012Metric, F.Cu at (182.9, 126.9)
- added C64: 0.1uF, Capacitor_SMD:C_0402_1005Metric, F.Cu at (191.9, 122.5)
- added C65: 0.1uF, Capacitor_SMD:C_0402_1005Metric, F.Cu at (191.9, 124.5)
- added C66: 1uF, Capacitor_SMD:C_0402_1005Metric, F.Cu at (191.9, 126.4)
- added C67: 0.1uF, Capacitor_SMD:C_0402_1005Metric, F.Cu at (191.9, 128.4)
- added C68: 0.1uF, Capacitor_SMD:C_0201_0603Metric, F.Cu at (181.9, 109.3)
- added C69: 33pF, Capacitor_SMD:C_0201_0603Metric, F.Cu at (181.9, 111.0)
- added C70: 33pF, Capacitor_SMD:C_0201_0603Metric, F.Cu at (181.9, 112.8)
- added C71: 33pF, Capacitor_SMD:C_0201_0603Metric, F.Cu at (181.9, 114.5)
- added C72: 0.1uF, Capacitor_SMD:C_0201_0603Metric, B.Cu at (167.6, 120.9)
- added C73: 8.2pF, Capacitor_SMD:C_0201_0603Metric, F.Cu at (181.9, 118.0)
- added C74: 100pF, Capacitor_SMD:C_0201_0603Metric, F.Cu at (181.9, 119.8)
- added C75: 0.1uF, Capacitor_SMD:C_0201_0603Metric, B.Cu at (166.1, 120.9)
- added C76: 8.2pF, Capacitor_SMD:C_0201_0603Metric, F.Cu at (184.3, 109.3)
- added C77: 100pF, Capacitor_SMD:C_0201_0603Metric, F.Cu at (184.3, 111.0)
- added C78: 8.2pF, Capacitor_SMD:C_0201_0603Metric, F.Cu at (184.3, 112.8)
- added C79: 100pF, Capacitor_SMD:C_0201_0603Metric, F.Cu at (184.3, 114.5)
- added D2: WS2812B-2020, pcs_lib:LED_WS2812B-2020_PLCC4_2.0x2.0mm, B.Cu at (168.4, 92.7)
- added D4: WS2812B-2020, pcs_lib:LED_WS2812B-2020_PLCC4_2.0x2.0mm, B.Cu at (168.4, 95.2)
- added D5: WS2812B-2020, pcs_lib:LED_WS2812B-2020_PLCC4_2.0x2.0mm, B.Cu at (136.4, 97.8)
- added D6: WS2812B-2020, pcs_lib:LED_WS2812B-2020_PLCC4_2.0x2.0mm, B.Cu at (168.4, 97.8)
- added J1: VBUS_IN, pcs_lib:CONN_SD-43650-005_02_MOL, F.Cu at (137.2, 121.9)
- added J2: Motor1, pcs_lib:TE_2-1445100-3, F.Cu at (143.5, 95.7)
- added R14: 100k, Resistor_SMD:R_0402_1005Metric, B.Cu at (148.3, 98.3)
- added R15: 8.2k, Resistor_SMD:R_0201_0603Metric, B.Cu at (150.1, 98.3)
- added R16: 75k, Resistor_SMD:R_0201_0603Metric, B.Cu at (167.6, 116.3)
- added R21: 5.1k, Resistor_SMD:R_0201_0603Metric, B.Cu at (167.6, 115.6)
- added R23: 100k, Resistor_SMD:R_0402_1005Metric, B.Cu at (148.3, 100.3)
- added R24: 8.2k, Resistor_SMD:R_0201_0603Metric, B.Cu at (150.1, 100.3)
- added R27: 100k, Resistor_SMD:R_0402_1005Metric, B.Cu at (148.3, 102.4)
- added R28: 8.2k, Resistor_SMD:R_0201_0603Metric, B.Cu at (150.1, 102.4)
- added R3: 5.1k, Resistor_SMD:R_0201_0603Metric, B.Cu at (146.3, 115.0)
- added R4: 0R, Resistor_SMD:R_0201_0603Metric, B.Cu at (161.8, 138.4)
- added R43: 5.1k, Resistor_SMD:R_0201_0603Metric, F.Cu at (184.3, 116.3)
- added R44: 470Ω, Resistor_SMD:R_0201_0603Metric, F.Cu at (184.3, 118.0)
- added R45: 470Ω, Resistor_SMD:R_0201_0603Metric, F.Cu at (184.3, 119.8)
- added R46: 470Ω, Resistor_SMD:R_0201_0603Metric, F.Cu at (184.3, 121.5)
- added R47: 100k, Resistor_SMD:R_0402_1005Metric, F.Cu at (194.8, 120.6)
- added R48: 8.2k, Resistor_SMD:R_0201_0603Metric, F.Cu at (186.8, 109.3)
- added R49: 75k, Resistor_SMD:R_0201_0603Metric, B.Cu at (167.6, 120.1)
- added R50: 100R, Resistor_SMD:R_0201_0603Metric, B.Cu at (153.9, 95.5)
- added R51: 100R, Resistor_SMD:R_0201_0603Metric, B.Cu at (153.9, 94.0)
- added R52: 100R, Resistor_SMD:R_0201_0603Metric, B.Cu at (153.9, 92.5)
- added R53: 100R, Resistor_SMD:R_0201_0603Metric, B.Cu at (153.9, 96.3)
- added R54: 5.1k, Resistor_SMD:R_0201_0603Metric, B.Cu at (167.6, 119.4)
- added R55: 2.2k, Resistor_SMD:R_0201_0603Metric, B.Cu at (153.9, 97.0)
- added R56: 100k, Resistor_SMD:R_0402_1005Metric, F.Cu at (194.8, 122.5)
- added R57: 8.2k, Resistor_SMD:R_0201_0603Metric, F.Cu at (189.2, 109.3)
- added R58: 2.2k, Resistor_SMD:R_0201_0603Metric, B.Cu at (153.9, 93.2)
- added R59: 2.2k, Resistor_SMD:R_0201_0603Metric, B.Cu at (153.9, 94.7)
- added R60: 100k, Resistor_SMD:R_0402_1005Metric, F.Cu at (194.8, 124.5)
- added R61: 8.2k, Resistor_SMD:R_0201_0603Metric, F.Cu at (189.2, 114.5)
- added R8: 0R, Resistor_SMD:R_0201_0603Metric, B.Cu at (169.2, 100.3)
- added U12: DRV8316C, pcs_lib:QFN-40_EP_5x7_Pitch0.5mm, F.Cu at (157.5, 109.2)
- added U13: TPS2553DBVR, pcs_lib:SOT-23-6_TI_DBV0006A, F.Cu at (167.6, 120.0)
- added U14: TPD4E05U06DQA, Package_SON:USON-10_2.5x1.0mm_P0.5mm, B.Cu at (156.5, 96.0)
- added U4: TPS2553DBVR, pcs_lib:SOT-23-6_TI_DBV0006A, F.Cu at (167.6, 116.2)
- added Y1: 25MHz, Crystal:Crystal_SMD_SeikoEpson_FA128-4Pin_2.0x1.6mm, F.Cu at (160.3, 138.4)
- C1, C2, C41, C53, D1, R1, R2: moved to B.Cu
- C10: renamed from C8; moved to B.Cu
- C11: renamed from C9; moved to B.Cu
- C12: renamed from C10; moved to B.Cu
- C13: renamed from C11; moved to B.Cu
- C14: renamed from C12; moved to B.Cu
- C15: renamed from C13; moved to B.Cu
- C16: renamed from C14; moved to B.Cu
- C21: renamed from C16; moved to B.Cu
- C22: renamed from C17; moved to B.Cu
- C25: renamed from C19; moved to B.Cu
- C28: renamed from C22; moved to B.Cu
- C29: renamed from C23; moved to B.Cu
- C30: renamed from C24; moved to B.Cu
- C31: renamed from C25; moved to B.Cu
- C32: renamed from C26; moved to B.Cu
- C33: renamed from C27; moved to B.Cu
- C34: renamed from C28; moved to B.Cu
- C4: renamed from C3; moved to B.Cu
- C44: value 22uF -> 8.2pF; footprint Capacitor_SMD:C_0603_1608Metric -> Capacitor_SMD:C_0201_0603Metric; moved to B.Cu
- C45: value 47nF -> 100pF; footprint Capacitor_SMD:C_0402_1005Metric -> Capacitor_SMD:C_0201_0603Metric; moved to B.Cu
- C46: renamed from C32; moved to B.Cu
- C47: renamed from C33; moved to B.Cu
- C49: renamed from C35; moved to B.Cu
- C50: renamed from C36; moved to B.Cu
- C51: renamed from C37; moved to B.Cu
- C52: renamed from C38; moved to B.Cu
- C54: renamed from C39; moved to B.Cu
- C55: renamed from C40; moved to B.Cu
- C56: renamed from C42; moved to B.Cu
- C57: renamed from C43; moved to B.Cu
- C6: renamed from C4; moved to B.Cu
- C7: renamed from C5; moved to B.Cu
- C8: renamed from C6; moved to B.Cu
- C9: renamed from C7; moved to B.Cu
- D3: renamed from D2; moved to B.Cu
- D7: renamed from D3; moved to B.Cu
- J3: value 2-1445100-3 -> Motor2
- J4: value Encoder -> Encoder1
- J5: value 436500212 -> Encoder2; footprint pcs_lib:CONN_SD-43650-005_02_MOL -> Connector_Molex:Molex_PicoBlade_53261-0671_1x06-1MP_P1.25mm_Horizontal; moved to B.Cu
- R10: renamed from R7; moved to B.Cu
- R11: renamed from R8; moved to B.Cu
- R12: renamed from R9; moved to B.Cu
- R13: renamed from R10; moved to B.Cu
- R17: renamed from R11; moved to B.Cu
- R18: renamed from R12; moved to B.Cu
- R19: renamed from R13; moved to B.Cu
- R20: renamed from R14; moved to B.Cu
- R22: renamed from R15; moved to B.Cu
- R25: renamed from R16; moved to B.Cu
- R26: renamed from R17; moved to B.Cu
- R29: renamed from R18; moved to B.Cu
- R30: renamed from R19; moved to B.Cu
- R32: renamed from R21; moved to B.Cu
- R33: renamed from R22; moved to B.Cu
- R34: renamed from R23; moved to B.Cu
- R35: renamed from R24; moved to B.Cu
- R36: renamed from R25; moved to B.Cu
- R37: renamed from R26; moved to B.Cu
- R38: renamed from R27; moved to B.Cu
- R40: value 2.2k -> 27k; moved to B.Cu
- R41: value 2.2k -> 5.1k; moved to B.Cu
- R42: value 2.2k -> 22Ω; footprint Resistor_SMD:R_0201_0603Metric -> Resistor_SMD:R_0402_1005Metric
- R5: renamed from R3; moved to B.Cu
- R6: renamed from R4; moved to B.Cu
- R7: renamed from R5; moved to B.Cu
- SW2: value MCU Reset -> USR_BTN1
- TP1: renamed from TP3; value 5V0_VSENSE -> EXT_RGB_DIN; moved to B.Cu
- TP2: renamed from TP1; value 5V0_VSENSE -> nRST
- TP4: renamed from TP5; moved to B.Cu
- TP7: renamed from TP8; moved to B.Cu
- U11: value TPD4E05U06DQA -> TPS2553DBVR; footprint Package_SON:USON-10_2.5x1.0mm_P0.5mm -> pcs_lib:SOT-23-6_TI_DBV0006A
- U5: renamed from U4; moved to B.Cu
- moved C53 91.9 mm to (167.6, 124.7)
- moved C45 86.2 mm to (150.1, 103.4)
- moved D7 82.8 mm to (136.4, 113.3), turned to -90 degrees
- moved C1 81.2 mm to (137.2, 134.3), turned to 180 degrees
- moved C2 81.0 mm to (137.2, 135.9)
- moved C57 80.8 mm to (138.7, 108.0), turned to -90 degrees
- moved U1 80.0 mm to (144.1, 137.2)
- moved C55 79.2 mm to (140.0, 108.0), turned to 90 degrees
- moved C29 77.6 mm to (144.3, 105.4), turned to 90 degrees
- moved R39 77.1 mm to (136.4, 113.3), turned to 90 degrees
- moved U10 77.0 mm to (139.2, 108.0)
- moved U9 76.1 mm to (139.2, 113.3)
- moved C32 75.7 mm to (143.0, 109.0), turned to 180 degrees
- moved R1 75.7 mm to (143.0, 135.1), turned to -90 degrees
- moved C17 75.3 mm to (135.6, 93.0), turned to -90 degrees
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- renumbered C15 to C17, C20 to C26, C21 to C27, C29 to C35, C30 to C36, C31 to C37, C34 to C48, J8 to J10, J9 to J11, J10 to J12, J11 to J13, J1 to J6, J2 to J7, J6 to J8, J7 to J9, R20 to R31, R28 to R39, R6 to R9, TP4 to TP3, TP6 to TP5, TP7 to TP6, TP9 to TP8, TP10 to TP9, U9 to U10, U5 to U6, U6 to U7, U7 to U8, U8 to U9
Connections:
- C41 pad 1: GND -> /driver1/5V_ENC_SW
- C41 pad 2: /power/3V3_VSENSE_AI -> GND
- C44 pad 1: Net-(U10-FB_BK) -> /driver1/OUTC
- C44 pad 2: GND -> /driver1/VSENSE_C_AI
- C45 pad 1: Net-(U10-CPL) -> /driver1/VSENSE_C_AI
- C45 pad 2: Net-(U10-CPH) -> GND
- C49 pad 1: /power/VBUS_ISENSE_AI -> /micro/VBUS_ISENSE_AI
- C50 pad 2: /power/5V0_VSENSE_AI -> /micro/5V0_VSENSE_AI
- C52 pad 2: /power/VBUS_VSENSE_AI -> /micro/VBUS_VSENSE_AI
- C53 pad 1: 3V3A -> 5V0
- D3 pad 1: Net-(D2-DOUT) -> Net-(D3-DOUT)
- J3 pad 1: /driver1/OUTA -> /driver2/OUTA
- J3 pad 2: /driver1/OUTB -> /driver2/OUTB
- J3 pad 3: /driver1/OUTC -> /driver2/OUTC
- J4 pad 1: Net-(J4-Pin_1) -> /driver1/EXT_ENC_A_MISO
- J4 pad 2: Net-(J4-Pin_2) -> /driver1/EXT_ENC_B_MOSI
- J4 pad 3: Net-(J4-Pin_3) -> /driver1/EXT_ENC_SCK
- J4 pad 4: Net-(J4-Pin_4) -> /driver1/EXT_ENC_Z_CS
- J4 pad 5: 5V0 -> /driver1/5V_ENC_SW
- J5 pad 1: /power/VBUS_IN -> /driver2/EXT_ENC_A_MISO
- J5 pad 2: GND -> /driver2/EXT_ENC_B_MOSI
- J5 pad 3: GND -> /driver2/EXT_ENC_SCK
- R17 pad 2: Net-(J4-Pin_1) -> /driver1/EXT_ENC_SCK
- R18 pad 2: Net-(J4-Pin_2) -> /driver1/EXT_ENC_B_MOSI
- R19 pad 2: Net-(J4-Pin_3) -> /driver1/EXT_ENC_A_MISO
- R20 pad 2: Net-(J4-Pin_4) -> /driver1/EXT_ENC_Z_CS
- R22 pad 2: Net-(J4-Pin_4) -> /driver1/EXT_ENC_Z_CS
- R25 pad 2: Net-(J4-Pin_3) -> /driver1/EXT_ENC_A_MISO
- R26 pad 2: Net-(J4-Pin_2) -> /driver1/EXT_ENC_B_MOSI
- R32 pad 2: /power/VBUS_ISENSE_AI -> /micro/VBUS_ISENSE_AI
- R33 pad 1: /power/5V0_VSENSE_AI -> /micro/5V0_VSENSE_AI
- R34 pad 2: /power/5V0_VSENSE_AI -> /micro/5V0_VSENSE_AI
- R37 pad 1: /power/VBUS_VSENSE_AI -> /micro/VBUS_VSENSE_AI
- R38 pad 2: /power/VBUS_VSENSE_AI -> /micro/VBUS_VSENSE_AI
- R40 pad 1: 3V3 -> GND
- R40 pad 2: Net-(J13-Pin_4) -> Net-(U11-ILIM)
- R41 pad 2: Net-(J13-Pin_3) -> /micro/PWR_nFLT
- R42 pad 1: 3V3 -> Net-(U12-FB_BK)
- R42 pad 2: Net-(J13-Pin_2) -> Net-(U12-SW_BK)
- TP1 pad 1: Net-(D2-DOUT) -> /micro/EXT_RGB_DIN
- U11 pad 1: Net-(J13-Pin_4) -> 5V0
- U11 pad 2: Net-(J13-Pin_3) -> GND
- U11 pad 3: GND -> /micro/EXP_PWR_EN
- U11 pad 4: Net-(J13-Pin_2) -> /micro/PWR_nFLT
- U11 pad 5: Net-(J13-Pin_1) -> Net-(U11-ILIM)
- U11 pad 6: unconnected-(U11-NC-Pad6) -> EXP_5V0_SW
- U2 pad A2: unconnected-(U2-PC13-PadA2) -> /micro/USR_BTN1
- U2 pad A3: unconnected-(U2-PE2-PadA3) -> /driver1/DRV_INLA
- U2 pad A4: unconnected-(U2-PB9-PadA4) -> /micro/FDCAN1_TX
- U2 pad A5: unconnected-(U2-PB7-PadA5) -> /micro/EXP_I2C_SDA
- U2 pad A6: unconnected-(U2-PB4-PadA6) -> /driver1/ENC_A_MISO
- U2 pad A8: unconnected-(U2-PA15-PadA8) -> /micro/ECAT_SYNC0
- U2 pad B10: unconnected-(U2-PA12-PadB10) -> /micro/USB_P
- U2 pad B3: unconnected-(U2-PE3-PadB3) -> /driver1/DRV_INLB
- U2 pad B4: unconnected-(U2-PB8-PadB4) -> /micro/FDCAN1_RX
- U2 pad B5: unconnected-(U2-PB6-PadB5) -> /micro/EXP_I2C_SCL
- U2 pad B6: unconnected-(U2-PD5-PadB6) -> /driver2/DRV_nSLEEP
- U2 pad B7: unconnected-(U2-PD2-PadB7) -> /micro/ECAT_SYNC1
- U2 pad B8: unconnected-(U2-PC11-PadB8) -> /micro/QSPI_nCS
- U2 pad B9: unconnected-(U2-PC10-PadB9) -> /driver1/ENC_SCK
- U2 pad C1: unconnected-(U2-PH0-PadC1) -> /micro/RCC_OSC_IN
- U2 pad C10: unconnected-(U2-PA11-PadC10) -> /micro/USB_N
- U2 pad C3: unconnected-(U2-PE4-PadC3) -> /driver1/DRV_INLC
- U2 pad C4: unconnected-(U2-PE1-PadC4) -> /driver1/DRV_DRVOFF
- U2 pad C5: unconnected-(U2-PB5-PadC5) -> /driver1/ENC_B_MOSI
- U2 pad C6: unconnected-(U2-PD6-PadC6) -> /driver2/DRV_DRVOFF
- U2 pad C7: unconnected-(U2-PD3-PadC7) -> /driver2/ENC_SCK
- U2 pad C8: unconnected-(U2-PC12-PadC8) -> /driver1/ENC_EN
- U2 pad C9: unconnected-(U2-PA9-PadC9) -> /driver1/DRV_INHB
- U2 pad D1: unconnected-(U2-PH1-PadD1) -> /micro/RCC_OSC_OUT
- U2 pad D10: unconnected-(U2-PA10-PadD10) -> /driver1/DRV_INHC
- U2 pad D3: unconnected-(U2-PE5-PadD3) -> /micro/RGB_DIN
- U2 pad D4: unconnected-(U2-PE0-PadD4) -> /driver1/DRV_nSLEEP
- U2 pad D6: unconnected-(U2-PD7-PadD6) -> /micro/EXP_UART_DE
- U2 pad D7: unconnected-(U2-PD4-PadD7) -> /driver2/DRV_nSCS
- U2 pad D8: unconnected-(U2-PD0-PadD8) -> /micro/EXP_PWR_EN
- U2 pad D9: unconnected-(U2-PA8-PadD9) -> /driver1/DRV_INHA
- U2 pad E10: unconnected-(U2-PC7-PadE10) -> /driver2/DRV_INHB
- U2 pad E2: unconnected-(U2-PC2_C-PadE2) -> /micro/VBUS_VSENSE_AI
- U2 pad E3: unconnected-(U2-PE6-PadE3) -> /micro/ECAT_nRST
- U2 pad E8: unconnected-(U2-PD1-PadE8) -> /micro/ECAT_IRQ
- U2 pad E9: unconnected-(U2-PC9-PadE9) -> /driver1/ENC_Z_CS
- U2 pad F1: unconnected-(U2-PC0-PadF1) -> /driver1/ISENSE_C_AI
- U2 pad F10: unconnected-(U2-PC6-PadF10) -> /driver2/DRV_INHA
- U2 pad F2: unconnected-(U2-PC1-PadF2) -> /driver2/ISENSE_C_AI
- U2 pad F3: unconnected-(U2-PC3_C-PadF3) -> /micro/VBUS_ISENSE_AI
- U2 pad F9: unconnected-(U2-PC8-PadF9) -> /driver2/DRV_INHC
- U2 pad G10: unconnected-(U2-PB15-PadG10) -> /driver2/ENC_B_MOSI
- U2 pad G2: unconnected-(U2-PA0-PadG2) -> /driver1/VSENSE_A_AI
- U2 pad G3: unconnected-(U2-PA4-PadG3) -> /driver2/ISENSE_A_AI
- U2 pad G4: unconnected-(U2-PC4-PadG4) -> /driver2/VSENSE_C_AI
- U2 pad G5: unconnected-(U2-PB2-PadG5) -> /micro/QSPI_CLK
- U2 pad G6: unconnected-(U2-PE10-PadG6) -> /micro/QSPI_IO3
- U2 pad G7: unconnected-(U2-PE14-PadG7) -> /DRV_SDI
- U2 pad G8: unconnected-(U2-PD15-PadG8) -> /driver2/ENC_Z_CS
- U2 pad G9: unconnected-(U2-PD11-PadG9) -> /micro/PWR_nFLT
- U2 pad H10: unconnected-(U2-PB14-PadH10) -> /driver2/ENC_A_MISO
- U2 pad H2: unconnected-(U2-PA1-PadH2) -> /driver1/VSENSE_B_AI
- U2 pad H3: unconnected-(U2-PA5-PadH3) -> /driver1/VSENSE_C_AI
- U2 pad H4: unconnected-(U2-PC5-PadH4) -> /micro/5V0_VSENSE_AI
- U2 pad H5: unconnected-(U2-PE7-PadH5) -> /micro/QSPI_IO0
- U2 pad H6: unconnected-(U2-PE11-PadH6) -> /driver1/DRV_nSCS
- U2 pad H7: unconnected-(U2-PE15-PadH7) -> /driver1/DRV_nFAULT
- U2 pad H8: unconnected-(U2-PD14-PadH8) -> /driver2/ENC_EN
- U2 pad H9: unconnected-(U2-PD10-PadH9) -> /driver2/DRV_INLC
- U2 pad J10: unconnected-(U2-PD13-PadJ10) -> /driver2/ENC_B_MOSI
- U2 pad J2: unconnected-(U2-PA2-PadJ2) -> /driver1/ISENSE_A_AI
- U2 pad J3: unconnected-(U2-PA6-PadJ3) -> /driver2/DRV_nFAULT
- U2 pad J4: unconnected-(U2-PB0-PadJ4) -> /driver2/VSENSE_A_AI
- U2 pad J5: unconnected-(U2-PE8-PadJ5) -> /micro/QSPI_IO1
- U2 pad J6: unconnected-(U2-PE12-PadJ6) -> /DRV_SCLK
- U2 pad J7: unconnected-(U2-PB10-PadJ7) -> /micro/EXP_UART_TX
- U2 pad J8: unconnected-(U2-PB13-PadJ8) -> /micro/FDCAN2_TX
- U2 pad J9: unconnected-(U2-PD9-PadJ9) -> /driver2/DRV_INLB
- U2 pad K10: unconnected-(U2-PD12-PadK10) -> /driver2/ENC_A_MISO
- U2 pad K2: unconnected-(U2-PA3-PadK2) -> /driver1/ISENSE_B_AI
- U2 pad K3: unconnected-(U2-PA7-PadK3) -> /driver2/ISENSE_B_AI
- U2 pad K4: unconnected-(U2-PB1-PadK4) -> /driver2/VSENSE_B_AI
- U2 pad K5: unconnected-(U2-PE9-PadK5) -> /micro/QSPI_IO2
- U2 pad K6: unconnected-(U2-PE13-PadK6) -> /DRV_SDO
- U2 pad K7: unconnected-(U2-PB11-PadK7) -> /micro/EXP_UART_RX
- U2 pad K8: unconnected-(U2-PB12-PadK8) -> /micro/FDCAN2_RX
- U2 pad K9: unconnected-(U2-PD8-PadK9) -> /driver2/DRV_INLA
- U3 pad 33: /driver1/DRV_SDO -> /DRV_SDO
- U3 pad 34: /driver1/DRV_SDI -> /DRV_SDI
- U3 pad 35: /driver1/DRV_SCLK -> /DRV_SCLK
- U5 pad 1: Net-(J4-Pin_4) -> /driver1/EXT_ENC_A_MISO
- U5 pad 10: unconnected-(U4-NC-Pad10) -> /driver1/EXT_ENC_A_MISO
- U5 pad 2: Net-(J4-Pin_3) -> /driver1/EXT_ENC_B_MOSI
- U5 pad 4: Net-(J4-Pin_2) -> /driver1/EXT_ENC_SCK
- U5 pad 5: Net-(J4-Pin_1) -> /driver1/EXT_ENC_Z_CS
- U5 pad 6: unconnected-(U4-NC-Pad6) -> /driver1/EXT_ENC_Z_CS
- U5 pad 7: unconnected-(U4-NC-Pad7) -> /driver1/EXT_ENC_SCK
- U5 pad 9: unconnected-(U4-NC-Pad9) -> /driver1/EXT_ENC_B_MOSI
Routing:
- net (no net): vias 0 -> 2
Other:
- copper layers 2 -> 6
