File: hw/stm32h7/eth.kicad_sch (KiCad schematic)
At the start: 5 parts, among them J10 miniPCIe, J6 RJ45_Hanrun_HR911105A_Horizon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, J7 RJ45_Hanrun_HR911105A_Horizon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, J8 FDCAN2, J9 FDCAN1

Commit message: WIP: H7 schematic and PCB layout progress
Parts:
- renumbered J8 to J10, J9 to J11, J10 to J12, J6 to J8, J7 to J9
Changed lines of the file:
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@@
 		(in_pos_files yes)
 		(dnp no)
-		(property "Reference" "J9"
+		(property "Reference" "J11"
 			(at 279.4 189.484 0)
 			(show_name no)
@@
 			(project "pcs_bldc_h7"
 				(path "/5fd46c36-5bf8-4b01-84ef-7a32553f026d/2667a4f0-e40e-4a6c-bdeb-6f94afb25317"
-					(reference "J9")
+					(reference "J11")
 					(unit 1)
 				)
@@
 		(in_pos_files yes)
 		(dnp no)
-		(property "Reference" "J8"
+		(property "Reference" "J10"
 			(at 278.13 207.264 0)
 			(show_name no)
@@
 			(project "pcs_bldc_h7"
 				(path "/5fd46c36-5bf8-4b01-84ef-7a32553f026d/2667a4f0-e40e-4a6c-bdeb-6f94afb25317"
-					(reference "J8")
+					(reference "J10")
 					(unit 1)
 				)
@@
 		(dnp no)
 		(fields_autoplaced yes)
-		(property "Reference" "J10"
+		(property "Reference" "J12"
 			(at 287.02 96.52 0)
 			(show_name no)
@@
 			(project "pcs_bldc_h7"
 				(path "/5fd46c36-5bf8-4b01-84ef-7a32553f026d/2667a4f0-e40e-4a6c-bdeb-6f94afb25317"
-					(reference "J10")
+					(reference "J12")
 					(unit 1)
 				)
@@
 		(dnp no)
 		(fields_autoplaced yes)
-		(property "Reference" "J7"
+		(property "Reference" "J9"
 			(at 168.91 177.8 0)
 			(show_name no)
@@
 			(project "pcs_bldc_h7"
 				(path "/5fd46c36-5bf8-4b01-84ef-7a32553f026d/2667a4f0-e40e-4a6c-bdeb-6f94afb25317"
-					(reference "J7")
+					(reference "J9")
 					(unit 1)
 				)
@@
 		(dnp no)
 		(fields_autoplaced yes)
-		(property "Reference" "J6"
+		(property "Reference" "J8"
 			(at 167.64 138.43 0)
 			(show_name no)
@@
 			(project "pcs_bldc_h7"
 				(path "/5fd46c36-5bf8-4b01-84ef-7a32553f026d/2667a4f0-e40e-4a6c-bdeb-6f94afb25317"
-					(reference "J6")
+					(reference "J8")
 					(unit 1)
 				)
