File: hw/stm32h7/ex_comms.kicad_sch (KiCad schematic)
At the start: 3 parts, among them J11 Bus_PCI_Express_Mini

Commit message: WIP: H7 schematic and PCB layout progress
Parts:
- renumbered J11 to J13
Other:
- moved on the sheet: FID1, FID2, J13
