File: hw/stm32h7/pcs_bldc_h7.kicad_sch (KiCad schematic)
At the start: 0 parts

Commit message: WIP: schematic bringup
Other:
- sheet driver1 ports: added DRV_DRVOFF, DRV_INHA, DRV_INHB, DRV_INHC, DRV_INLA, DRV_INLB, DRV_INLC, DRV_SCLK, DRV_SDI, DRV_SDO, DRV_nFAULT, DRV_nSCS, DRV_nSLEEP, ENC_A_MISO, ENC_B_MOSI, ENC_EN, ENC_SCK, ENC_SW_nFLT, ENC_Z_CS, ISENSE_A_AI, ISENSE_B_AI, ISENSE_C_AI, VSENSE_A_AI, VSENSE_B_AI, VSENSE_C_AI; removed none
- sheet driver2 ports: added DRV_DRVOFF, DRV_INHA, DRV_INHB, DRV_INHC, DRV_INLA, DRV_INLB, DRV_INLC, DRV_SCLK, DRV_SDI, DRV_SDO, DRV_nFAULT, DRV_nSCS, DRV_nSLEEP, ENC_A_MISO, ENC_B_MOSI, ENC_EN, ENC_SCK, ENC_SW_nFLT, ENC_Z_CS, ISENSE_A_AI, ISENSE_B_AI, ISENSE_C_AI, VSENSE_A_AI, VSENSE_B_AI, VSENSE_C_AI; removed none
- sheet micro ports: added ENCODER_1; removed none
- sheet power ports: added 5V0_VSENSE_AI, VBUS_ISENSE_AI, VBUS_VSENSE_AI; removed none

Commit message: WIP: H7 schematic and PCB layout progress
Parts:
- added J1: VBUS_IN, pcs_lib:CONN_SD-43650-005_02_MOL, symbol pcs_bldc_sym_lib:436500212
- added J2: Motor1, pcs_lib:TE_2-1445100-3, symbol pcs_bldc_sym_lib:2-1445100-3
- added J3: Motor2, pcs_lib:TE_2-1445100-3, symbol pcs_bldc_sym_lib:2-1445100-3
- added J4: Encoder1, Connector_Molex:Molex_PicoBlade_53261-0671_1x06-1MP_P1.25mm_Horizontal, symbol Connector:Conn_01x06_Socket
- added J5: Encoder2, Connector_Molex:Molex_PicoBlade_53261-0671_1x06-1MP_P1.25mm_Horizontal, symbol Connector:Conn_01x06_Socket
Connections:
- new net GND: J1.2, J1.3 (shield), J2.4 (SHIELD), J2.5 (SHIELD), J3.4 (SHIELD), J3.5 (SHIELD), J4.6 (Pin_6), J5.6 (Pin_6)
- new net driver1/5V_ENC_SW: J4.5 (Pin_5)
- new net driver1/EXT_ENC_A_MISO: J4.1 (Pin_1)
- new net driver1/EXT_ENC_B_MOSI: J4.2 (Pin_2)
- new net driver1/EXT_ENC_SCK: J4.3 (Pin_3)
- new net driver1/EXT_ENC_Z_CS: J4.4 (Pin_4)
- new net driver1/OUTA: J2.1
- new net driver1/OUTB: J2.2
- new net driver1/OUTC: J2.3
- new net driver2/5V_ENC_SW: J5.5 (Pin_5)
- new net driver2/EXT_ENC_A_MISO: J5.1 (Pin_1)
- new net driver2/EXT_ENC_B_MOSI: J5.2 (Pin_2)
- new net driver2/EXT_ENC_SCK: J5.3 (Pin_3)
- new net driver2/EXT_ENC_Z_CS: J5.4 (Pin_4)
- new net driver2/OUTA: J3.1
- new net driver2/OUTB: J3.2
- new net driver2/OUTC: J3.3
- new net power/VBUS_IN: J1.1
Other:
- sheet driver1 ports: added 5V_ENC_SW, EXT_ENC_A_MISO, EXT_ENC_B_MOSI, EXT_ENC_SCK, EXT_ENC_Z_CS, OUTA, OUTB, OUTC; removed none
- sheet driver2 ports: added 5V_ENC_SW, EXT_ENC_A_MISO, EXT_ENC_B_MOSI, EXT_ENC_SCK, EXT_ENC_Z_CS, OUTA, OUTB, OUTC; removed none
- sheet micro ports: added 5V0_VSENSE_AI, DRV1_DRVOFF, DRV1_INLA, DRV1_INLB, DRV1_INLC, DRV1_ISENSE_A_AI, DRV1_ISENSE_B_AI, DRV1_ISENSE_C_AI, DRV1_PWM_1, DRV1_PWM_2, DRV1_PWM_3, DRV1_VSENSE_A_AI, DRV1_VSENSE_B_AI, DRV1_VSENSE_C_AI, DRV1_nCS, DRV1_nFAULT, DRV1_nSLEEP, DRV2_DRVOFF, DRV2_INLA, DRV2_INLB, DRV2_INLC, DRV2_ISENSE_A_AI, DRV2_ISENSE_B_AI, DRV2_ISENSE_C_AI, DRV2_PWM_1, DRV2_PWM_2, DRV2_PWM_3, DRV2_VSENSE_A_AI, DRV2_VSENSE_B_AI, DRV2_VSENSE_C_AI, DRV2_nCS, DRV2_nFAULT, DRV2_nSLEEP, DRV_SCLK, DRV_SDI, DRV_SDO, ENC1_A_MISO, ENC1_B_MOSI, ENC1_EN, ENC1_SCK, ENC1_SW_nFLT, ENC1_Z_CS, ENC2_A_MISO, ENC2_B_MOSI, ENC2_EN, ENC2_SCK, ENC2_SW_nFLT, ENC2_Z_CS, EXP_PWR_EN, EXP_PWR_nFLT, VBUS_ISENSE_AI, VBUS_VSENSE_AI; removed ENCODER_1
- sheet power ports: added EXP_PWR_EN, EXP_PWR_nFLT, VBUS_IN; removed none
